File: ExoFlexV2/ExoFlex_Kicad.kicad_pcb (KiCad board)
At the start: 2 copper layers, 101.6 x 53.3 mm, 13 parts, among them J1 Power, J2 PWM, J3 Analog, J4 PWM, J5 Analog, J6 Communication, J7 Digital

Commit message: Many changes
Debouncing, power protection, potentiometer limits, etc.
Parts:
- added C10: 1uF, Capacitor_SMD:C_0603_1608Metric, F.Cu at (312.9, -72.0)
- added C100: 0,01uF, Capacitor_SMD:C_0603_1608Metric, F.Cu at (269.7, -45.1)
- added C101: 0,01uF, Capacitor_SMD:C_0603_1608Metric, F.Cu at (269.7, -42.6)
- added C107: 0,1uF, Capacitor_SMD:C_0603_1608Metric, F.Cu at (294.3, -56.2)
- added C108: 0,1uF, Capacitor_SMD:C_0603_1608Metric, F.Cu at (298.3, -58.7)
- added C109: 0,1uF, Capacitor_SMD:C_0603_1608Metric, F.Cu at (290.3, -58.7)
- added C11: 47uF, Capacitor_SMD:C_0603_1608Metric, F.Cu at (316.9, -69.5)
- added C110: 0,1uF, Capacitor_SMD:C_0603_1608Metric, F.Cu at (290.3, -56.2)
- added C111: 0,1uF, Capacitor_SMD:C_0603_1608Metric, F.Cu at (298.3, -56.2)
- added C112: 0,1uF, Capacitor_SMD:C_0603_1608Metric, F.Cu at (294.3, -58.7)
- added C113: 0,01uF, Capacitor_SMD:C_0603_1608Metric, F.Cu at (296.3, -67.0)
- added C114: 0,01uF, Capacitor_SMD:C_0603_1608Metric, F.Cu at (300.3, -72.0)
- added C115: 0,01uF, Capacitor_SMD:C_0603_1608Metric, F.Cu at (292.3, -72.0)
- added C116: 0,01uF, Capacitor_SMD:C_0603_1608Metric, F.Cu at (304.4, -69.5)
- added C117: 0,01uF, Capacitor_SMD:C_0603_1608Metric, F.Cu at (304.4, -67.0)
- added C118: 0,01uF, Capacitor_SMD:C_0603_1608Metric, F.Cu at (304.4, -72.0)
- added C120: 0,01uF, Capacitor_SMD:C_0603_1608Metric, F.Cu at (292.3, -69.5)
- added C121: 0,01uF, Capacitor_SMD:C_0603_1608Metric, F.Cu at (296.3, -69.5)
- added C122: 0,01uF, Capacitor_SMD:C_0603_1608Metric, F.Cu at (300.3, -67.0)
- added C123: 0,01uF, Capacitor_SMD:C_0603_1608Metric, F.Cu at (292.3, -67.0)
- added C124: 0,01uF, Capacitor_SMD:C_0603_1608Metric, F.Cu at (296.3, -72.0)
- added C125: 0,01uF, Capacitor_SMD:C_0603_1608Metric, F.Cu at (300.3, -69.5)
- added C17: 1 uF, Capacitor_SMD:C_0603_1608Metric, F.Cu at (256.4, -72.0)
- added C18: 47 nF, Capacitor_SMD:C_0603_1608Metric, F.Cu at (248.4, -72.0)
- added C19: 3,3 nF, Capacitor_SMD:C_0603_1608Metric, F.Cu at (256.4, -64.5)
- added C20: 1 uF, Capacitor_SMD:C_0603_1608Metric, F.Cu at (248.4, -69.5)
- added C21: 47 nF, Capacitor_SMD:C_0603_1608Metric, F.Cu at (260.4, -72.0)
- added C22: 3,3 nF, Capacitor_SMD:C_0603_1608Metric, F.Cu at (256.4, -69.5)
- added C23: 47 nF, Capacitor_SMD:C_0603_1608Metric, F.Cu at (256.4, -67.0)
- added C24: 3,3 nF, Capacitor_SMD:C_0603_1608Metric, F.Cu at (260.4, -67.0)
- added C25: 3,3 nF, Capacitor_SMD:C_0603_1608Metric, F.Cu at (252.4, -72.0)
- added C26: 47 nF, Capacitor_SMD:C_0603_1608Metric, F.Cu at (252.4, -69.5)
- added C27: 3,3 nF, Capacitor_SMD:C_0603_1608Metric, F.Cu at (248.4, -67.0)
- added C28: 3,3 nF, Capacitor_SMD:C_0603_1608Metric, F.Cu at (248.4, -64.5)
- added C29: 47 nF, Capacitor_SMD:C_0603_1608Metric, F.Cu at (252.4, -67.0)
- added C3: 0,047uF, Capacitor_SMD:C_0603_1608Metric, F.Cu at (316.9, -72.0)
- added C30: 3,3 nF, Capacitor_SMD:C_0603_1608Metric, F.Cu at (252.4, -64.5)
- added C31: 3,3 nF, Capacitor_SMD:C_0603_1608Metric, F.Cu at (260.4, -69.5)
- added C32: 1uF, Capacitor_SMD:C_0603_1608Metric, F.Cu at (286.1, -42.6)
- added C33: 1uF, Capacitor_SMD:C_0603_1608Metric, F.Cu at (286.1, -45.1)
- added C34: 1uF, Capacitor_SMD:C_0603_1608Metric, F.Cu at (290.1, -45.1)
- added C35: 0,01uF, Capacitor_SMD:C_0603_1608Metric, F.Cu at (256.4, -55.5)
- added C36: 0,01uF, Capacitor_SMD:C_0603_1608Metric, F.Cu at (256.4, -58.0)
- added C37: 0,01uF, Capacitor_SMD:C_0603_1608Metric, F.Cu at (248.4, -55.5)
- added C38: 0,01uF, Capacitor_SMD:C_0603_1608Metric, F.Cu at (260.4, -58.0)
- added C39: 0,01uF, Capacitor_SMD:C_0603_1608Metric, F.Cu at (260.4, -55.5)
- added C40: 0,01uF, Capacitor_SMD:C_0603_1608Metric, F.Cu at (252.4, -55.5)
- added C41: 0,1uF, Capacitor_SMD:C_0603_1608Metric, F.Cu at (252.4, -58.0)
- added C42: 0,01uF, Capacitor_SMD:C_0603_1608Metric, F.Cu at (248.4, -50.4)
- added C43: 0,01uF, Capacitor_SMD:C_0603_1608Metric, F.Cu at (248.4, -58.0)
- added C44: 0,01uF, Capacitor_SMD:C_0603_1608Metric, F.Cu at (256.4, -52.9)
- added C45: 0,01uF, Capacitor_SMD:C_0603_1608Metric, F.Cu at (252.4, -52.9)
- added C46: 0,01uF, Capacitor_SMD:C_0603_1608Metric, F.Cu at (248.4, -52.9)
- added C47: 0,01uF, Capacitor_SMD:C_0603_1608Metric, F.Cu at (252.4, -50.4)
- added C51: 0,1uF, Capacitor_SMD:C_0603_1608Metric, F.Cu at (309.7, -59.1)
- added C52: 0,1uF, Capacitor_SMD:C_0603_1608Metric, F.Cu at (305.7, -56.6)
- added C53: 0,1uF, Capacitor_SMD:C_0603_1608Metric, F.Cu at (305.7, -59.1)
- added C54: 0,1uF, Capacitor_SMD:C_0603_1608Metric, F.Cu at (309.7, -56.6)
- added C55: 0,1uF, Capacitor_SMD:C_0603_1608Metric, F.Cu at (252.4, -37.2)
- added C56: 0,01uF, Capacitor_SMD:C_0603_1608Metric, F.Cu at (252.4, -39.7)
- added C57: 0,01uF, Capacitor_SMD:C_0603_1608Metric, F.Cu at (256.4, -44.7)
- added C58: 0,01uF, Capacitor_SMD:C_0603_1608Metric, F.Cu at (248.4, -44.7)
- added C59: 0,01uF, Capacitor_SMD:C_0603_1608Metric, F.Cu at (260.4, -42.2)
- added C6: 0,047uF, Capacitor_SMD:C_0603_1608Metric, F.Cu at (312.9, -69.5)
- added C60: 0,01uF, Capacitor_SMD:C_0603_1608Metric, F.Cu at (248.4, -39.7)
- added C61: 0,01uF, Capacitor_SMD:C_0603_1608Metric, F.Cu at (248.4, -42.2)
- added C62: 0,01uF, Capacitor_SMD:C_0603_1608Metric, F.Cu at (256.4, -42.2)
- added C63: 0,01uF, Capacitor_SMD:C_0603_1608Metric, F.Cu at (252.4, -42.2)
- added C64: 0,01uF, Capacitor_SMD:C_0603_1608Metric, F.Cu at (256.4, -39.7)
- added C65: 0,01uF, Capacitor_SMD:C_0603_1608Metric, F.Cu at (252.4, -44.7)
- added C66: 0,01uF, Capacitor_SMD:C_0603_1608Metric, F.Cu at (248.4, -37.2)
- added C67: 0,01uF, Capacitor_SMD:C_0603_1608Metric, F.Cu at (260.4, -44.7)
- added C68: 0,01uF, Capacitor_SMD:C_0603_1608Metric, F.Cu at (273.7, -58.0)
- added C69: 0,01uF, Capacitor_SMD:C_0603_1608Metric, F.Cu at (269.7, -58.0)
- added C70: 0,01uF, Capacitor_SMD:C_0603_1608Metric, F.Cu at (281.7, -52.9)
- added C71: 0,01uF, Capacitor_SMD:C_0603_1608Metric, F.Cu at (281.7, -58.0)
- added C72: 0,01uF, Capacitor_SMD:C_0603_1608Metric, F.Cu at (269.7, -52.9)
- added C73: 0,01uF, Capacitor_SMD:C_0603_1608Metric, F.Cu at (277.7, -58.0)
- added C74: 0,01uF, Capacitor_SMD:C_0603_1608Metric, F.Cu at (277.7, -52.9)
- added C75: 0,01uF, Capacitor_SMD:C_0603_1608Metric, F.Cu at (273.7, -55.5)
- added C76: 0,01uF, Capacitor_SMD:C_0603_1608Metric, F.Cu at (281.7, -55.5)
- added C77: 0,01uF, Capacitor_SMD:C_0603_1608Metric, F.Cu at (277.7, -55.5)
- added C78: 0,01uF, Capacitor_SMD:C_0603_1608Metric, F.Cu at (269.7, -55.5)
- added C79: 0,01uF, Capacitor_SMD:C_0603_1608Metric, F.Cu at (273.7, -52.9)
- added C80: 0,01uF, Capacitor_SMD:C_0603_1608Metric, F.Cu at (279.0, -69.5)
- added C81: 0,01uF, Capacitor_SMD:C_0603_1608Metric, F.Cu at (283.1, -69.5)
- added C82: 0,01uF, Capacitor_SMD:C_0603_1608Metric, F.Cu at (271.0, -72.0)
- added C83: 0,01uF, Capacitor_SMD:C_0603_1608Metric, F.Cu at (275.0, -69.5)
- added C84: 0,01uF, Capacitor_SMD:C_0603_1608Metric, F.Cu at (271.0, -67.0)
- added C85: 0,01uF, Capacitor_SMD:C_0603_1608Metric, F.Cu at (275.0, -72.0)
- added C86: 0,01uF, Capacitor_SMD:C_0603_1608Metric, F.Cu at (271.0, -64.5)
- added C87: 0,01uF, Capacitor_SMD:C_0603_1608Metric, F.Cu at (279.0, -72.0)
- added C88: 0,01uF, Capacitor_SMD:C_0603_1608Metric, F.Cu at (271.0, -69.5)
- added C89: 0,1uF, Capacitor_SMD:C_0603_1608Metric, F.Cu at (275.0, -67.0)
- added C90: 0,01uF, Capacitor_SMD:C_0603_1608Metric, F.Cu at (283.1, -72.0)
- added C91: 0,01uF, Capacitor_SMD:C_0603_1608Metric, F.Cu at (279.0, -67.0)
- added C92: 0,01uF, Capacitor_SMD:C_0603_1608Metric, F.Cu at (275.0, -64.5)
- added C95: 0,1uF, Capacitor_SMD:C_0603_1608Metric, F.Cu at (277.7, -45.1)
- added C96: 0,1uF, Capacitor_SMD:C_0603_1608Metric, F.Cu at (273.7, -42.6)
- added C97: 0,1uF, Capacitor_SMD:C_0603_1608Metric, F.Cu at (269.7, -40.1)
- added C98: 0,01uF, Capacitor_SMD:C_0603_1608Metric, F.Cu at (273.7, -40.1)
- added C99: 0,01uF, Capacitor_SMD:C_0603_1608Metric, F.Cu at (273.7, -45.1)
- added J10: Conn_01x03_Male, Connector_PinHeader_2.54mm:PinHeader_1x03_P2.54mm_Vertical, F.Cu at (144.2, -44.7)
- added J11: Conn_01x04_Male, Connector_PinHeader_2.54mm:PinHeader_1x04_P2.54mm_Vertical, F.Cu at (143.5, -68.4)
- added J12: Conn_01x03_Male, Connector_PinHeader_2.54mm:PinHeader_1x03_P2.54mm_Vertical, F.Cu at (148.5, -68.4)
- added J13: Conn_01x03_Male, Connector_PinHeader_2.54mm:PinHeader_1x03_P2.54mm_Vertical, F.Cu at (139.4, -48.1)
- added J14: Conn_01x03_Male, Connector_PinHeader_2.54mm:PinHeader_1x03_P2.54mm_Vertical, F.Cu at (134.2, -58.7)
- added J15: Conn_01x04_Male, Connector_PinHeader_2.54mm:PinHeader_1x04_P2.54mm_Vertical, F.Cu at (144.2, -54.4)
- added J16: Conn_01x09_Male, Connector_PinHeader_2.54mm:PinHeader_1x09_P2.54mm_Vertical, F.Cu at (134.2, -68.4)
- added J17: Conn_01x08_Male, Connector_PinHeader_2.54mm:PinHeader_1x08_P2.54mm_Vertical, F.Cu at (138.9, -68.4)
- added J18: Conn_01x04_Male, Connector_PinHeader_2.54mm:PinHeader_1x04_P2.54mm_Vertical, F.Cu at (148.8, -54.4)
- added J19: Conn_01x09_Male, Connector_PinHeader_2.54mm:PinHeader_1x09_P2.54mm_Vertical, F.Cu at (129.6, -58.7)
- added J8: Conn_01x03_Male, Connector_PinHeader_2.54mm:PinHeader_1x03_P2.54mm_Vertical, F.Cu at (149.5, -42.0)
- added J9: Conn_01x03_Male, Connector_PinHeader_2.54mm:PinHeader_1x03_P2.54mm_Vertical, F.Cu at (138.9, -58.7)
- added K1: UD2-5NU, FootPrint:UD2_NU_KEM-L, F.Cu at (87.1, -60.5)
- added R1: 1,5k, Resistor_SMD:R_0603_1608Metric, F.Cu at (193.7, -74.5)
- added R10: R_Small_US, Resistor_SMD:R_0603_1608Metric, F.Cu at (180.7, -71.7)
- added R11: R_Small_US, Resistor_SMD:R_0603_1608Metric, F.Cu at (184.7, -74.2)
- added R12: R_Small_US, Resistor_SMD:R_0603_1608Metric, F.Cu at (189.5, -65.4)
- added R13: 5k, Resistor_SMD:R_0603_1608Metric, F.Cu at (193.5, -67.9)
- added R14: 5k, Resistor_SMD:R_0603_1608Metric, F.Cu at (189.5, -67.9)
- added R15: 5k, Resistor_SMD:R_0603_1608Metric, F.Cu at (180.9, -50.1)
- added R16: R_Small_US, Resistor_SMD:R_0603_1608Metric, F.Cu at (180.9, -45.1)
- added R17: R_Small_US, Resistor_SMD:R_0603_1608Metric, F.Cu at (180.9, -47.6)
- added R18: R_Small_US, Resistor_SMD:R_0603_1608Metric, F.Cu at (184.9, -50.1)
- added R19: R_Small_US, Resistor_SMD:R_0603_1608Metric, F.Cu at (193.4, -47.6)
- added R2: 1,1k, Resistor_SMD:R_0603_1608Metric, F.Cu at (189.7, -74.5)
- added R20: R_Small_US, Resistor_SMD:R_0603_1608Metric, F.Cu at (189.4, -50.1)
- added R21: R_Small_US, Resistor_SMD:R_0603_1608Metric, F.Cu at (193.3, -43.3)
- added R22: R_Small_US, Resistor_SMD:R_0603_1608Metric, F.Cu at (193.4, -50.1)
- added R23: R_Small_US, Resistor_SMD:R_0603_1608Metric, F.Cu at (189.4, -47.6)
- added R24: R_Small_US, Resistor_SMD:R_0603_1608Metric, F.Cu at (189.3, -43.3)
- added R25: R_Small_US, Resistor_SMD:R_0603_1608Metric, F.Cu at (193.4, -37.7)
- added R26: R_Small_US, Resistor_SMD:R_0603_1608Metric, F.Cu at (180.8, -57.0)
- added R27: R_Small_US, Resistor_SMD:R_0603_1608Metric, F.Cu at (189.4, -37.7)
- added R28: R_Small_US, Resistor_SMD:R_0603_1608Metric, F.Cu at (180.8, -59.5)
- added R29: R_Small_US, Resistor_SMD:R_0603_1608Metric, F.Cu at (189.4, -40.2)
- added R3: 6,8k, Resistor_SMD:R_0603_1608Metric, F.Cu at (189.7, -72.0)
- added R30: R_Small_US, Resistor_SMD:R_0603_1608Metric, F.Cu at (184.8, -59.5)
- added R31: R_Small_US, Resistor_SMD:R_0603_1608Metric, F.Cu at (193.4, -40.2)
- added R32: R_Small_US, Resistor_SMD:R_0603_1608Metric, F.Cu at (180.8, -54.5)
- added R33: R_Small_US, Resistor_SMD:R_0603_1608Metric, F.Cu at (184.8, -57.0)
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Connections:
- net /*2 renamed /STM SIGNALS/D53
- net /*3 renamed /STM SIGNALS/A2
- net /*4 renamed /STM SIGNALS/D52
- net /*52 renamed /STM SIGNALS/AGND
- net /*6 renamed /STM SIGNALS/D51
- net /22 renamed /STM SIGNALS/D34
- net /23 renamed /STM SIGNALS/D35
- net /25 renamed /STM SIGNALS/D36
- net /27 renamed /STM SIGNALS/D37
- net /29 renamed /STM SIGNALS/D38
- net /30 renamed /STM SIGNALS/D31
- net /31 renamed /STM SIGNALS/D39
- net /32 renamed /STM SIGNALS/D30
- net /33 renamed /STM SIGNALS/D40
- net /34 renamed /STM SIGNALS/D29
- net /36 renamed /STM SIGNALS/D28
- net /37 renamed /STM SIGNALS/D41
- net /39 renamed /STM SIGNALS/D42
- net /40 renamed /STM SIGNALS/D27
- net /42 renamed /STM SIGNALS/D26
- net /A10 renamed /STM SIGNALS/D17
- net /A11 renamed /STM SIGNALS/D14
- net /A12 renamed /STM SIGNALS/D18
- net /A13 renamed /STM SIGNALS/AREF
- net /A14 renamed /STM SIGNALS/D19
- net /A8 renamed /STM SIGNALS/D16
- net /IOREF renamed Net-(F1-Pad1)
- net /RX0/0 renamed /STM SIGNALS/D54
- net /RX1/19 renamed /STM SIGNALS/D45
- net /RX2/17 renamed /STM SIGNALS/D44
- net /RX3/15 renamed /STM SIGNALS/D43
- net /TX1/18 renamed /STM SIGNALS/NRST
- net /TX2/16 renamed /STM SIGNALS/IOREF
- net /TX3/14 renamed /STM SIGNALS/NC
- J1 pad 1: unconnected-(J1-Pad1) -> +5V
- J2 pad 1: /SCL/21 -> +5V
- J2 pad 2: /SDA/20 -> Net-(F2-Pad1)
- J3 pad 1: /A0 -> Net-(J3-Pad1)
- J3 pad 2: /A1 -> +5V
- J4 pad 1: /*7 -> TOR_MOT_3
- J4 pad 3: /*5 -> MOT_ENC_1
- J4 pad 7: /TX0/1 -> MOT_ENC_2
- J5 pad 2: /A9 -> BUT_PROX_SEC
- J5 pad 8: /A15 -> +5V
- J6 pad 7: /SDA/20 -> +3V3
- J6 pad 8: /SCL/21 -> /STM SIGNALS/D46
- J7 pad 1: GND -> /STM SIGNALS/VDDA
- J7 pad 10: /47 -> SW5
- J7 pad 11: /*44 -> MAG3_POT_OUT
- J7 pad 12: /*45 -> PROX_1
- J7 pad 14: /43 -> PROX_2
- J7 pad 16: /41 -> PROX_3
- J7 pad 17: /38 -> +5V
- J7 pad 2: GND -> SW1
- J7 pad 22: /35 -> +5V
- J7 pad 27: /28 -> +5V
- J7 pad 29: /26 -> MAG_AMP_4
- J7 pad 31: /24 -> TOR_MOT_2
- J7 pad 4: /53 -> SW2
- J7 pad 5: /50 -> +5V
- J7 pad 6: /51 -> SW3
- J7 pad 7: /48 -> MAG_AMP_1
- J7 pad 8: /49 -> SW4
- J7 pad 9: /*46 -> MAG_AMP_2
Other:
- board size 101.6 x 53.3 mm -> 53.3 x 101.6 mm

Commit message: quque truc
Parts:
- removed U42, U43: ADCMP602BRMZ, FootPrint:ADCMP602BRMZ
- added C1: 150uF 50V, FootPrint:CAP_EEHZS1H151P, F.Cu at (334.9, -67.1)
- added C102: 0,01uF, Capacitor_SMD:C_0603_1608Metric, F.Cu at (375.2, -61.8)
- added C103: 0,01uF, Capacitor_SMD:C_0603_1608Metric, F.Cu at (375.2, -66.8)
- added C104: 0,01uF, Capacitor_SMD:C_0603_1608Metric, F.Cu at (387.2, -71.8)
- added C105: 10 uF, Capacitor_SMD:C_0603_1608Metric, F.Cu at (383.2, -66.8)
- added C106: 10 uF, Capacitor_SMD:C_0603_1608Metric, F.Cu at (391.2, -69.3)
- added C119: 10 uF, Capacitor_SMD:C_0603_1608Metric, F.Cu at (377.3, -34.9)
- added C12: 10uF, Capacitor_SMD:C_0603_1608Metric, F.Cu at (356.0, -62.0)
- added C126: 1nF, Capacitor_SMD:C_0603_1608Metric, F.Cu at (368.4, -41.2)
- added C127: 1nF, Capacitor_SMD:C_0603_1608Metric, F.Cu at (364.4, -36.1)
- added C128: 1nF, Capacitor_SMD:C_0603_1608Metric, F.Cu at (372.4, -37.4)
- added C129: 0,01uF, Capacitor_SMD:C_0603_1608Metric, F.Cu at (377.4, -45.0)
- added C13: 10uF, Capacitor_SMD:C_0603_1608Metric, F.Cu at (360.8, -65.0)
- added C130: 0,01uF, Capacitor_SMD:C_0603_1608Metric, F.Cu at (333.8, -30.1)
- added C131: 0,01uF, Capacitor_SMD:C_0603_1608Metric, F.Cu at (341.8, -32.6)
- added C132: 0,01uF, Capacitor_SMD:C_0603_1608Metric, F.Cu at (345.8, -37.4)
- added C133: 0,01uF, Capacitor_SMD:C_0603_1608Metric, F.Cu at (341.8, -30.1)
- added C134: 0,01uF, Capacitor_SMD:C_0603_1608Metric, F.Cu at (345.3, -42.5)
- added C135: 0,1uF, Capacitor_SMD:C_0603_1608Metric, F.Cu at (341.3, -37.6)
- added C136: 0,01uF, Capacitor_SMD:C_0603_1608Metric, F.Cu at (337.8, -35.1)
- added C137: 0,01uF, Capacitor_SMD:C_0603_1608Metric, F.Cu at (348.8, -45.0)
- added C138: 0,01uF, Capacitor_SMD:C_0603_1608Metric, F.Cu at (329.8, -35.2)
- added C139: 0,01uF, Capacitor_SMD:C_0603_1608Metric, F.Cu at (273.5, -86.9)
- added C14: 10uF, Capacitor_SMD:C_0603_1608Metric, F.Cu at (356.8, -68.5)
- added C140: 0,01uF, Capacitor_SMD:C_0603_1608Metric, F.Cu at (269.5, -86.9)
- added C141: 0,01uF, Capacitor_SMD:C_0603_1608Metric, F.Cu at (281.5, -91.8)
- added C15: 10uF, Capacitor_SMD:C_0603_1608Metric, F.Cu at (356.8, -65.9)
- added C16: 10uF, Capacitor_SMD:C_0603_1608Metric, F.Cu at (356.0, -59.4)
- added C2: 10 uF, Capacitor_SMD:C_0805_2012Metric, F.Cu at (344.4, -51.7)
- added C4: 100uF 20V, FootPrint:CAP_PC_8X7_NCH, F.Cu at (348.1, -58.2)
- added C48: 1nF, Capacitor_SMD:C_0603_1608Metric, F.Cu at (391.6, -41.6)
- added C49: 0,1uF, Capacitor_SMD:C_0603_1608Metric, F.Cu at (387.6, -41.6)
- added C5: 220uF 50V, FootPrint:CAP_EEHZS1H221P, F.Cu at (334.9, -55.3)
- added C50: 0,01uF, Capacitor_SMD:C_0603_1608Metric, F.Cu at (387.6, -39.1)
- added C7: 100uF, Capacitor_SMD:C_1210_3225Metric, F.Cu at (364.0, -70.9)
- added C8: 220uF 20V, FootPrint:CAP_20SVPK220M, F.Cu at (348.4, -68.1)
- added C9: 10uF, Capacitor_SMD:C_0603_1608Metric, F.Cu at (360.8, -67.6)
- added C93: 0,01uF, Capacitor_SMD:C_0603_1608Metric, F.Cu at (383.2, -61.8)
- added C94: 0,01uF, Capacitor_SMD:C_0603_1608Metric, F.Cu at (379.2, -69.3)
- added D1: TPD1E, FootPrint:DPY2_TEX, F.Cu at (186.4, -22.9)
- added D10: TPD1E, FootPrint:DPY2_TEX, F.Cu at (48.0, -95.4)
- added D11: TPD1E, FootPrint:DPY2_TEX, F.Cu at (39.7, -102.4)
- added D12: TPD1E, FootPrint:DPY2_TEX, F.Cu at (53.5, -90.6)
- added D13: TPD1E, FootPrint:DPY2_TEX, F.Cu at (48.0, -93.0)
- added D14: TPD1E, FootPrint:DPY2_TEX, F.Cu at (36.9, -97.7)
- added D15: TPD1E, FootPrint:DPY2_TEX, F.Cu at (42.4, -102.4)
- added D16: TPD1E, FootPrint:DPY2_TEX, F.Cu at (56.2, -100.1)
- added D17: TPD1E, FootPrint:DPY2_TEX, F.Cu at (53.5, -95.4)
- added D18: TPD1E, FootPrint:DPY2_TEX, F.Cu at (36.9, -90.6)
- added D19: TPD1E, FootPrint:DPY2_TEX, F.Cu at (42.4, -90.6)
- added D2: DSS12UTR, FootPrint:SODFL3618X110N, F.Cu at (71.8, -102.4)
- added D20: TPD1E, FootPrint:DPY2_TEX, F.Cu at (50.7, -90.6)
- added D21: TPD1E, FootPrint:DPY2_TEX, F.Cu at (56.2, -93.0)
- added D22: TPD1E, FootPrint:DPY2_TEX, F.Cu at (39.7, -97.7)
- added D23: TPD1E, FootPrint:DPY2_TEX, F.Cu at (64.5, -102.4)
- added D24: TPD1E, FootPrint:DPY2_TEX, F.Cu at (42.4, -93.0)
- added D25: TPD1E, FootPrint:DPY2_TEX, F.Cu at (61.8, -100.1)
- added D26: TPD1E, FootPrint:DPY2_TEX, F.Cu at (45.2, -102.4)
- added D27: TPD1E, FootPrint:DPY2_TEX, F.Cu at (36.9, -95.4)
- added D28: TPD1E, FootPrint:DPY2_TEX, F.Cu at (42.4, -95.4)
- added D29: TPD1E, FootPrint:DPY2_TEX, F.Cu at (53.5, -102.4)
- added D3: TPD1E, FootPrint:DPY2_TEX, F.Cu at (358.3, -71.4)
- added D30: TPD1E, FootPrint:DPY2_TEX, F.Cu at (59.0, -97.7)
- added D31: TPD1E, FootPrint:DPY2_TEX, F.Cu at (48.0, -88.3)
- added D32: TPD1E, FootPrint:DPY2_TEX, F.Cu at (50.7, -93.0)
- added D33: TPD1E, FootPrint:DPY2_TEX, F.Cu at (36.9, -88.3)
- added D34: TPD1E, FootPrint:DPY2_TEX, F.Cu at (53.5, -100.1)
- added D35: TPD1E, FootPrint:DPY2_TEX, F.Cu at (50.7, -95.4)
- added D36: TPD1E, FootPrint:DPY2_TEX, F.Cu at (39.7, -93.0)
- added D37: TPD1E, FootPrint:DPY2_TEX, F.Cu at (50.7, -100.1)
- added D38: TPD1E, FootPrint:DPY2_TEX, F.Cu at (48.0, -90.6)
- added D39: TPD1E, FootPrint:DPY2_TEX, F.Cu at (56.2, -95.4)
- added D4: TPD1E, FootPrint:DPY2_TEX, F.Cu at (45.2, -95.4)
- added D40: TPD1E, FootPrint:DPY2_TEX, F.Cu at (50.7, -102.4)
- added D41: TPD1E, FootPrint:DPY2_TEX, F.Cu at (61.8, -102.4)
- added D42: TPD1E, FootPrint:DPY2_TEX, F.Cu at (36.9, -93.0)
- added D43: TPD1E, FootPrint:DPY2_TEX, F.Cu at (48.0, -97.7)
- added D44: TPD1E, FootPrint:DPY2_TEX, F.Cu at (50.7, -88.3)
- added D45: TPD1E, FootPrint:DPY2_TEX, F.Cu at (56.2, -102.4)
- added D46: TPD1E, FootPrint:DPY2_TEX, F.Cu at (53.5, -93.0)
- added D47: TPD1E, FootPrint:DPY2_TEX, F.Cu at (53.5, -97.7)
- added D48: TPD1E, FootPrint:DPY2_TEX, F.Cu at (39.7, -88.3)
- added D49: TPD1E, FootPrint:DPY2_TEX, F.Cu at (59.0, -100.1)
- added D5: TPD1E, FootPrint:DPY2_TEX, F.Cu at (48.0, -100.1)
- added D50: TPD1E, FootPrint:DPY2_TEX, F.Cu at (42.4, -100.1)
- added D51: TPD1E, FootPrint:DPY2_TEX, F.Cu at (45.2, -97.7)
- added D52: TPD1E, FootPrint:DPY2_TEX, F.Cu at (48.0, -102.4)
- added D53: TPD1E, FootPrint:DPY2_TEX, F.Cu at (45.2, -88.3)
- added D54: TPD1E, FootPrint:DPY2_TEX, F.Cu at (61.8, -97.7)
- added D55: TPD1E, FootPrint:DPY2_TEX, F.Cu at (45.2, -93.0)
- added D56: TPD1E, FootPrint:DPY2_TEX, F.Cu at (36.9, -102.4)
- added D57: TPD1E, FootPrint:DPY2_TEX, F.Cu at (56.2, -97.7)
- added D58: TPD1E, FootPrint:DPY2_TEX, F.Cu at (42.4, -97.7)
- added D59: TPD1E, FootPrint:DPY2_TEX, F.Cu at (59.0, -102.4)
- added D6: TPD1E, FootPrint:DPY2_TEX, F.Cu at (59.0, -95.4)
- added D60: TPD1E, FootPrint:DPY2_TEX, F.Cu at (39.7, -100.1)
- added D61: TPD1E, FootPrint:DPY2_TEX, F.Cu at (39.7, -90.6)
- added D62: TPD1E, FootPrint:DPY2_TEX, F.Cu at (39.7, -95.4)
- added D63: TPD1E, FootPrint:DPY2_TEX, F.Cu at (36.9, -100.1)
- added D7: TPD1E, FootPrint:DPY2_TEX, F.Cu at (45.2, -100.1)
- added D8: TPD1E, FootPrint:DPY2_TEX, F.Cu at (42.4, -88.3)
- added D9: TPD1E, FootPrint:DPY2_TEX, F.Cu at (45.2, -90.6)
- added F1: SP5X20 16A, FootPrint:696108003002, F.Cu at (175.7, -104.2)
- added F2: FSF5X20 630mA, FootPrint:696108003002, F.Cu at (175.7, -115.3)
- added R100: 0 ohm, Resistor_SMD:R_0603_1608Metric, F.Cu at (329.8, -30.2)
- added R101: 15k, Resistor_SMD:R_0603_1608Metric, F.Cu at (333.8, -35.1)
- added R102: 15k, Resistor_SMD:R_0603_1608Metric, F.Cu at (277.5, -86.8)
- added R103: 15k, Resistor_SMD:R_0603_1608Metric, F.Cu at (281.5, -86.8)
- added R104: 0 ohm, Resistor_SMD:R_0603_1608Metric, F.Cu at (277.5, -89.3)
- added R105: 0 ohm, Resistor_SMD:R_0603_1608Metric, F.Cu at (277.0, -94.3)
- added R106: 0 ohm, Resistor_SMD:R_0603_1608Metric, F.Cu at (285.0, -94.3)
- added R107: 0 ohm, Resistor_SMD:R_0603_1608Metric, F.Cu at (281.0, -94.3)
- added R108: 0 ohm, Resistor_SMD:R_0603_1608Metric, F.Cu at (269.5, -89.5)
- added R109: 0 ohm, Resistor_SMD:R_0603_1608Metric, F.Cu at (281.5, -89.3)
- added R110: 15k, Resistor_SMD:R_0603_1608Metric, F.Cu at (285.5, -91.8)
- added R111: 15k, Resistor_SMD:R_0603_1608Metric, F.Cu at (273.5, -89.5)
- added R112: 15k, Resistor_SMD:R_0603_1608Metric, F.Cu at (277.5, -91.8)
- added R55: 220k, Resistor_SMD:R_0603_1608Metric, F.Cu at (402.0, -71.8)
- added R56: 2M, Resistor_SMD:R_0603_1608Metric, F.Cu at (410.0, -69.3)
- added R57: 2M, Resistor_SMD:R_0603_1608Metric, F.Cu at (402.0, -66.8)
- added R58: 2M, Resistor_SMD:R_0603_1608Metric, F.Cu at (406.0, -71.8)
- added R59: 430k, Resistor_SMD:R_0603_1608Metric, F.Cu at (406.0, -66.8)
- added R60: 430k, Resistor_SMD:R_0603_1608Metric, F.Cu at (410.0, -71.8)
- added R61: 430k, Resistor_SMD:R_0603_1608Metric, F.Cu at (402.0, -69.3)
- added R62: 2M, Resistor_SMD:R_0603_1608Metric, F.Cu at (410.0, -66.8)
- added R63: 2M, Resistor_SMD:R_0603_1608Metric, F.Cu at (406.0, -69.3)
- added R64: 2M, Resistor_SMD:R_0603_1608Metric, F.Cu at (383.2, -64.3)
- added R65: R_Small_US, Resistor_SMD:R_0603_1608Metric, F.Cu at (391.2, -71.8)
- added R66: R_Small_US, Resistor_SMD:R_0603_1608Metric, F.Cu at (387.2, -69.3)
- added R67: R_Small_US, Resistor_SMD:R_0603_1608Metric, F.Cu at (375.2, -69.3)
- added R68: R_Small_US, Resistor_SMD:R_0603_1608Metric, F.Cu at (383.2, -71.8)
- added R69: 0 ohm, Resistor_SMD:R_0603_1608Metric, F.Cu at (375.2, -71.8)
- added R70: 0 ohm, Resistor_SMD:R_0603_1608Metric, F.Cu at (379.2, -71.8)
- added R71: 0 ohm, Resistor_SMD:R_0603_1608Metric, F.Cu at (379.2, -61.8)
- added R72: R_Small_US, Resistor_SMD:R_0603_1608Metric, F.Cu at (379.2, -66.8)
- added R73: R_Small_US, Resistor_SMD:R_0603_1608Metric, F.Cu at (387.2, -64.3)
- added R74: 15k, Resistor_SMD:R_0603_1608Metric, F.Cu at (375.2, -64.3)
- added R75: 15k, Resistor_SMD:R_0603_1608Metric, F.Cu at (383.2, -69.3)
- added R76: 15k, Resistor_SMD:R_0603_1608Metric, F.Cu at (379.2, -64.3)
- added R77: 15k, Resistor_SMD:R_0603_1608Metric, F.Cu at (391.2, -66.8)
- added R78: 15k, Resistor_SMD:R_0603_1608Metric, F.Cu at (387.2, -66.8)
- added R79: 15k, Resistor_SMD:R_0603_1608Metric, F.Cu at (387.6, -52.9)
- added R80: 0 ohm, Resistor_SMD:R_0603_1608Metric, F.Cu at (391.6, -55.4)
- added R81: 5k, Resistor_SMD:R_0603_1608Metric, F.Cu at (387.6, -55.4)
- added R82: 5k, Resistor_SMD:R_0603_1608Metric, F.Cu at (387.6, -50.4)
- added R83: 15k, Resistor_SMD:R_0603_1608Metric, F.Cu at (368.4, -36.1)
- added R84: 15k, Resistor_SMD:R_0603_1608Metric, F.Cu at (376.5, -42.5)
- added R85: 15k, Resistor_SMD:R_0603_1608Metric, F.Cu at (364.4, -41.2)
- added R86: 15k, Resistor_SMD:R_0603_1608Metric, F.Cu at (368.4, -38.6)
- added R87: 15k, Resistor_SMD:R_0603_1608Metric, F.Cu at (372.4, -42.5)
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Connections:
- C10 pad 1: Net-(U4-Pad14) -> Net-(C10-Pad1)
- C10 pad 2: +5V -> +5VA
- C101 pad 1: +5VA -> +5V
- C107 pad 1: +5VA -> MAG_AMP_4
- C107 pad 2: +5V -> +5VA
- C108 pad 1: +5VA -> +5V
- C108 pad 2: +5V -> +5VA
- C109 pad 2: +5V -> +5VA
- C11 pad 2: +5V -> +5VA
- C110 pad 2: +5V -> +5VA
- C111 pad 2: +5V -> +5VA
- C112 pad 1: +5V -> +5VA
- C112 pad 2: +5V -> +5VA
- C117 pad 1: +5VA -> Net-(C117-Pad1)
- C118 pad 1: +5VA -> Net-(C118-Pad1)
- C120 pad 1: +5VA -> Net-(C120-Pad1)
- C121 pad 1: +5VA -> Net-(C121-Pad1)
- C122 pad 1: +5VA -> +5V
- C123 pad 1: +5VA -> TEMP_3
- C124 pad 1: +5VA -> TEMP_1
- C125 pad 1: +5VA -> TEMP_2
- C20 pad 1: +5V -> MAG_AMP_3
- C20 pad 2: +5V -> +5VA
- C21 pad 1: +5V -> MAG_AMP_2
- C21 pad 2: +5V -> +5VA
- C22 pad 1: +5V -> MAG_AMP_1
- C22 pad 2: +5V -> +5VA
- C23 pad 1: +5V -> MAG_LIM_1
- C23 pad 2: +5V -> +5VA
- C24 pad 1: +5V -> MAG_LIM_2
- C24 pad 2: +5V -> +5VA
- C25 pad 1: +5V -> MAG_AMP_3
- C25 pad 2: +5V -> +5VA
- C26 pad 1: +5V -> +5VA
- C26 pad 2: +5V -> +5VA
- C27 pad 1: +5V -> +5VA
- C27 pad 2: +5V -> +5VA
- C28 pad 1: +5V -> +5VA
- C28 pad 2: +5V -> +5VA
- C29 pad 1: +5V -> +5VA
- C29 pad 2: +5V -> +5VA
- C3 pad 2: +5V -> +5VA
- C30 pad 1: +5V -> +5VA
- C30 pad 2: +5V -> +5VA
- C31 pad 1: +5V -> +5VA
- C31 pad 2: +5V -> +5VA
- C32 pad 2: +5V -> +5VA
- C33 pad 1: +5V -> +5VA
- C33 pad 2: +5V -> +5VA
- C34 pad 1: +5V -> +5VA
- C34 pad 2: +5V -> +5VA
- C39 pad 1: +5VA -> Net-(C39-Pad1)
- C40 pad 1: +5VA -> Net-(C40-Pad1)
- C41 pad 1: +5V -> Net-(C41-Pad1)
- C42 pad 1: +5VA -> +5V
- C43 pad 1: +5VA -> MOT_ENC_2
- C44 pad 1: +5VA -> MOT_ENC_1
- C45 pad 1: +5VA -> MAG_LIM_1
- C46 pad 1: +5VA -> MAG_LIM_2
- C47 pad 1: +5VA -> MOT_ENC_3
- C51 pad 2: +5V -> +5VA
- C52 pad 2: +5V -> +5VA
- C53 pad 2: +5V -> +5VA
- C54 pad 1: +5V -> +5VA
- C54 pad 2: +5V -> +5VA
- C55 pad 1: +5V -> +5VA
- C6 pad 1: Net-(C7-Pad1) -> Net-(C6-Pad1)
- C6 pad 2: +5V -> +5VA
- C62 pad 1: +5VA -> Net-(C62-Pad1)
- C63 pad 1: +5VA -> Net-(C63-Pad1)
- C64 pad 1: +5VA -> Net-(C64-Pad1)
- C65 pad 1: +5VA -> LC_LIM_1
- C66 pad 1: +5VA -> LC_LIM_2
- C70 pad 1: +5VA -> LC_LIM_3
- C86 pad 1: +5VA -> TOR_MOT_2
- C87 pad 1: +5VA -> LC_LIM_1
- C88 pad 1: +5VA -> LC_LIM_2
- C89 pad 1: +5V -> TOR_MOT_3
- C90 pad 1: +5VA -> TOR_MOT_1
- C91 pad 1: +5VA -> LC_LIM_3
- C95 pad 1: +5V -> +5VA
- C95 pad 2: +5V -> +5VA
- C96 pad 1: +5V -> +5VA
- C96 pad 2: +5V -> +5VA
- C97 pad 1: +5V -> +5VA
- C97 pad 2: +5V -> +5VA
- J1 pad 1: +5V -> +5VA
- J10 pad 2: MAG_AMP_2 -> MAG_OUT_3
- J10 pad 3: +5V -> +5VA
- J11 pad 1: SWOUT1 -> +5VA
- J11 pad 2: SWOUT2 -> MAG_OUT_4
- J11 pad 3: SWOUT3 -> +5VA
- J12 pad 2: MAG3_POT_OUT -> LC_O+_1
- J12 pad 3: +5V -> +5VA
- J13 pad 2: MAG_AMP_2 -> LC_O+_2
- J13 pad 3: GND -> +5VA
- J14 pad 2: MAG_AMP_4 -> LC_O+_3
- J14 pad 3: +5V -> +5VA
- J16 pad 1: MAG1_POT1 -> SWOUT5
- J16 pad 2: MAG1_POT_OUT -> SWOUT6
- J16 pad 3: MAG1_POT2 -> SWOUT7
- J16 pad 4: MAG2_POT1 -> SWOUT8
- J18 pad 1: SWOUT5 -> MAG1_POT1
- J18 pad 2: SWOUT6 -> MAG1_POT_OUT
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
Commit message: Placement
Début du placement et modification d'après dernier review
Parts:
- removed C133, C134, C136, C137, C138, C139, C140, C141: 0,01uF, Capacitor_SMD:C_0603_1608Metric
- removed C135: 0,1uF, Capacitor_SMD:C_0603_1608Metric
- removed MH1, MH2, MH3, MH4, MH5, MH6: MountingHole_3.2mm, Arduino_MountingHole:MountingHole_3.2mm
- removed R100, R104, R105, R106, R107, R108, R109, R95, R98, R99: 0 ohm, Resistor_SMD:R_0603_1608Metric
- removed R101, R102, R103, R110, R111, R112: 15k, Resistor_SMD:R_0603_1608Metric
- removed R96, R97: 5k, Resistor_SMD:R_0603_1608Metric
- removed U39, U40, U41: ADCMP602BRMZ, FootPrint:ADCMP602BRMZ
- added CR1: 1SS321_LF, FootPrint:1SS321_LF, F.Cu at (180.6, 259.7)
- added CR2: TBAT54_LM, FootPrint:TBAT54_LM, F.Cu at (185.2, 259.5)
- added D64: TPD1E, FootPrint:DPY2_TEX, F.Cu at (41.8, 106.5)
- added D65: TPD1E, FootPrint:DPY2_TEX, F.Cu at (36.2, 173.4)
- added D66: TPD1E, FootPrint:DPY2_TEX, F.Cu at (19.7, 170.9)
- added D67: TPD1E, FootPrint:DPY2_TEX, F.Cu at (36.2, 170.9)
- added D68: TPD1E, FootPrint:DPY2_TEX, F.Cu at (19.7, 168.3)
- added D69: TPD1E, FootPrint:DPY2_TEX, F.Cu at (36.2, 168.3)
- added J20: AMP2, Connector_PinHeader_2.54mm:PinHeader_1x03_P2.54mm_Vertical, F.Cu at (38.8, 106.5)
- added TP100: 5005, FootPrint:KEYSTONE_5005, F.Cu at (140.5, 265.2)
- added TP101: 5005, FootPrint:KEYSTONE_5005, F.Cu at (150.0, 255.7)
- added TP102: 5005, FootPrint:KEYSTONE_5005, F.Cu at (103.5, 236.2)
- added TP103: 5005, FootPrint:KEYSTONE_5005, F.Cu at (94.0, 236.2)
- added TP104: 5005, FootPrint:KEYSTONE_5005, F.Cu at (84.5, 240.9)
- added TP105: 5005, FootPrint:KEYSTONE_5005, F.Cu at (79.8, 236.2)
- added TP106: 5005, FootPrint:KEYSTONE_5005, F.Cu at (89.3, 240.9)
- added TP107: 5005, FootPrint:KEYSTONE_5005, F.Cu at (89.3, 245.6)
- added TP108: 5005, FootPrint:KEYSTONE_5005, F.Cu at (79.8, 240.9)
- added TP109: 5005, FootPrint:KEYSTONE_5005, F.Cu at (94.0, 240.9)
- added TP110: 5005, FootPrint:KEYSTONE_5005, F.Cu at (84.5, 236.2)
- added TP111: 5005, FootPrint:KEYSTONE_5005, F.Cu at (89.3, 236.2)
- added TP112: 5005, FootPrint:KEYSTONE_5005, F.Cu at (84.5, 245.6)
- added TP113: 5005, FootPrint:KEYSTONE_5005, F.Cu at (98.7, 240.9)
- added TP114: 5005, FootPrint:KEYSTONE_5005, F.Cu at (79.8, 245.6)
- added TP115: 5005, FootPrint:KEYSTONE_5005, F.Cu at (94.0, 245.6)
- added TP116: 5005, FootPrint:KEYSTONE_5005, F.Cu at (98.7, 236.2)
- added TP117: 5005, FootPrint:KEYSTONE_5005, F.Cu at (162.0, 262.4)
- added TP118: 5005, FootPrint:KEYSTONE_5005, F.Cu at (171.4, 262.4)
- added TP119: 5005, FootPrint:KEYSTONE_5005, F.Cu at (166.7, 262.4)
- added TP120: 5005, FootPrint:KEYSTONE_5005, F.Cu at (170.4, 242.9)
- added TP121: 5005, FootPrint:KEYSTONE_5005, F.Cu at (184.6, 247.7)
- added TP122: 5005, FootPrint:KEYSTONE_5005, F.Cu at (179.9, 242.9)
- added TP123: 5005, FootPrint:KEYSTONE_5005, F.Cu at (184.6, 242.9)
- added TP124: 5005, FootPrint:KEYSTONE_5005, F.Cu at (175.1, 247.7)
- added TP125: 5005, FootPrint:KEYSTONE_5005, F.Cu at (170.4, 247.7)
- added TP126: 5005, FootPrint:KEYSTONE_5005, F.Cu at (165.7, 242.9)
- added TP127: 5005, FootPrint:KEYSTONE_5005, F.Cu at (179.9, 247.7)
- added TP128: 5005, FootPrint:KEYSTONE_5005, F.Cu at (165.7, 247.7)
- added TP129: 5005, FootPrint:KEYSTONE_5005, F.Cu at (175.1, 242.9)
- added TP130: 5005, FootPrint:KEYSTONE_5005, F.Cu at (127.3, 247.5)
- added TP91: 5005, FootPrint:KEYSTONE_5005, F.Cu at (140.5, 255.7)
- added TP92: 5005, FootPrint:KEYSTONE_5005, F.Cu at (140.5, 260.5)
- added TP93: 5005, FootPrint:KEYSTONE_5005, F.Cu at (145.2, 265.2)
- added TP94: 5005, FootPrint:KEYSTONE_5005, F.Cu at (145.2, 255.7)
- added TP95: 5005, FootPrint:KEYSTONE_5005, F.Cu at (150.0, 260.5)
- added TP96: 5005, FootPrint:KEYSTONE_5005, F.Cu at (150.0, 265.2)
- added TP97: 5005, FootPrint:KEYSTONE_5005, F.Cu at (154.7, 260.5)
- added TP98: 5005, FootPrint:KEYSTONE_5005, F.Cu at (154.7, 255.7)
- added TP99: 5005, FootPrint:KEYSTONE_5005, F.Cu at (145.2, 260.5)
- C101, C108: value 0,1uF -> 0,01uF
- C105: value 10 uF -> 0,1uF
- C106, C117, C118, C119, C120: value 10 uF -> 0,01uF
- C107, C62, C63, C64, C65, C86, C87, C88, C89: value 1nF -> 0,01uF
- C109, C50, C51, C52, C77, C92, C93, C94, C95: value 0,01uF -> 1nF
- C110, C111: value 0,01uF -> 10 uF
- C112, C53: value 0,01uF -> 0,1uF
- C122, C42: value 0,1uF -> 10 uF
- C123, C124, C125, C43, C44, C45: value 1nF -> 10 uF
- C126, C46: value 1nF -> 0,1uF
- C49, C67, C68, C69: value 0,1uF -> 1nF
- C71, C72, C73: value 1uF -> 0,1uF; moved to B.Cu
- C74, C75, C76: value 0,01uF -> 1uF; moved to B.Cu
- D2: value DSS12UTR -> SS12P2L-M3_86A; footprint FootPrint:SODFL3618X110N -> FootPrint:DIO_SS12P2L-M3_86A
- F1: value SP5X20 16A -> FSF5X20 200mA
- F2: value FSF5X20 630mA -> FSF5X20 500mA
- J10: value Conn_01x03_Male -> AMP_EVE1
- J11: value Conn_01x03_Male -> SWIVEL
- J12: value Conn_01x05_Male -> TOR_EXT1
- J13: value Conn_01x05_Male -> TOR_DOR1
- J14: value Conn_01x05_Male -> TOR_EVE1
- J15: value Conn_01x04_Male -> TOR_LIM; footprint Connector_PinHeader_2.54mm:PinHeader_1x04_P2.54mm_Vertical -> Connector_PinHeader_2.54mm:PinHeader_1x09_P2.54mm_Vertical
- J16: value Conn_01x04_Male -> AMP_LIM; footprint Connector_PinHeader_2.54mm:PinHeader_1x04_P2.54mm_Vertical -> Connector_PinHeader_2.54mm:PinHeader_1x09_P2.54mm_Vertical
- J17: value Conn_01x08_Male -> TOR2; footprint Connector_PinHeader_2.54mm:PinHeader_1x08_P2.54mm_Vertical -> Connector_PinHeader_2.54mm:PinHeader_1x03_P2.54mm_Vertical
- J18: value Conn_01x09_Male -> LIMITSWITCH; footprint Connector_PinHeader_2.54mm:PinHeader_1x09_P2.54mm_Vertical -> Connector_PinHeader_2.54mm:PinHeader_1x08_P2.54mm_Vertical
- J19: value Conn_01x09_Male -> PROXIMITY; footprint Connector_PinHeader_2.54mm:PinHeader_1x09_P2.54mm_Vertical -> Connector_PinHeader_2.54mm:PinHeader_1x08_P2.54mm_Vertical
- J4: value CN9 -> CN8; footprint Connector_PinSocket_2.54mm:PinSocket_2x15_P2.54mm_Vertical -> Connector_PinSocket_2.54mm:PinSocket_2x08_P2.54mm_Vertical
- J5: value CN8 -> CN9; footprint Connector_PinSocket_2.54mm:PinSocket_2x08_P2.54mm_Vertical -> Connector_PinSocket_2.54mm:PinSocket_2x15_P2.54mm_Vertical
- J8: value Conn_01x03_Male -> AMP_EXT1
- J9: value Conn_01x03_Male -> AMP_DOR1
- R11, R74, R85, R86, R87: value 15k -> 5k
- R12: value 15k -> 150
- R13: value 150 -> 3,6k
- R14: value 15k -> 2,5k
- R15: value 3,6k -> 7,5k
- R16: value 2,5k -> 7,5k
- R17, R18, R19, R33, R34, R35, R36, R46, R47, R75: value 15k -> 7,5k
- R20, R91: value 5k -> 7,5k
- R23, R24, R25, R26, R73: value R_Small_US -> 5k
- R27, R88, R89: value 0 ohm -> 5k
- R28, R29, R80, R90: value 0 ohm -> 0Ω
- R30, R37, R42, R43, R76, R77, R78, R79, R83, R84: value 15k -> 0Ω
- R31, R32, R41, R44, R45, R67, R68, R72: value R_Small_US -> 7,5k
- R38, R39, R40, R65, R66: value R_Small_US -> 0Ω
- R4: value 23,7 -> RE1C002UNTCL; footprint Resistor_SMD:R_0603_1608Metric -> FootPrint:DIO_RB558WMF_ROM
- R48: value 15k -> 10k
- R5: value 25,5k 1% -> 23,7
- R51: value 10k -> 220k
- R52: value 15k -> 220k
- R54, R55: value 220k -> 2M
- R57, R58: value 2M -> 430k
- R6: value 10k -> 25,5k 1%
- R60: value 430k -> 7,5k
- R61: value 430k -> 2M
- R64: value 2M -> 0Ω
- R69, R70, R71, R94: value 0 ohm -> 7,5k
- R7: value 2,5k -> 10k
- R8: value 5k -> 2,5k
- R81, R82: value 5k -> 0Ω
- R92, R93: value 5k -> 0 ohm
- U10: value SN74LV4T08PWR_V2 -> ADCMP602BRMZ; footprint FootPrint:SN74LV4T08PWR -> FootPrint:ADCMP602BRMZ
- U11: value SN74HC7032D_V2 -> ADCMP602BRMZ; footprint FootPrint:SN74HC7032D -> FootPrint:ADCMP602BRMZ
- U13: value ADCMP602BRMZ -> SN74LVC3G14DCUT_V2; footprint FootPrint:ADCMP602BRMZ -> FootPrint:SN74LVC3G14DCUT
- U14: value ADCMP602BRMZ -> SN74HC7032D_V2; footprint FootPrint:ADCMP602BRMZ -> FootPrint:SN74HC7032D
- U15: value SN74LVC3G14DCUT_V2 -> SN74LV4T08PWR_V2; footprint FootPrint:SN74LVC3G14DCUT -> FootPrint:SN74LV4T08PWR
- U16: value SN74LV4T08PWR_V2 -> SN74HC7032D_V2; footprint FootPrint:SN74LV4T08PWR -> FootPrint:SN74HC7032D
- U17: value SN74HC7032D_V2 -> 74LV244PW; footprint FootPrint:SN74HC7032D -> FootPrint:DB20
- U3: value LMZ23603TZ_NOPB -> CD4044BPWR; footprint FootPrint:LMZ23603 -> FootPrint:CD4044BPWR
- U38: value 74LV244PW -> ADCMP602BRMZ; footprint FootPrint:DB20 -> FootPrint:ADCMP602BRMZ
- U4: value CD4044BPWR -> LMZ23603TZ_NOPB; footprint FootPrint:CD4044BPWR -> FootPrint:LMZ23603
- U5: value SN74HC7032D_V2 -> TPS7A4701RGWR; footprint FootPrint:SN74HC7032D -> FootPrint:TPS7A470
- U6: value TPS7A4701RGWR -> SN74HC7032D_V2; footprint FootPrint:TPS7A470 -> FootPrint:SN74HC7032D
- U8: value SN74HC7032D_V2 -> SN74LV4T08PWR_V2; footprint FootPrint:SN74HC7032D -> FootPrint:SN74LV4T08PWR
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Connections:
- net Net-(F1-Pad1) renamed /POWER/24V_IN
- net Net-(J2-Pad2) renamed /POWER/5V_IN
- C1 pad 2: +5VA -> +5V
- C10 pad 2: +5VA -> +5V
- C100 pad 2: +5VA -> +5V
- C101 pad 1: +5V -> +5VA
- C101 pad 2: +5VA -> +5V
- C102 pad 2: +5VA -> +5V
- C103 pad 2: +5VA -> +5V
- C104 pad 2: +5VA -> +5V
- C105 pad 1: Net-(C105-Pad1) -> +5V
- C105 pad 2: +5VA -> +5V
- C106 pad 1: Net-(C106-Pad1) -> +5VA
- C106 pad 2: +5VA -> +5V
- C107 pad 1: MAG_AMP_4 -> +5VA
- C107 pad 2: +5VA -> +5V
- C108 pad 1: +5V -> +5VA
- C108 pad 2: +5VA -> +5V
- C109 pad 1: +5VA -> MAG_AMP_4
- C109 pad 2: +5VA -> +5V
- C11 pad 2: +5VA -> +5V
- C110 pad 1: +5VA -> Net-(C110-Pad1)
- C110 pad 2: +5VA -> +5V
- C111 pad 1: +5VA -> Net-(C111-Pad1)
- C111 pad 2: +5VA -> +5V
- C112 pad 1: +5VA -> +5V
- C112 pad 2: +5VA -> +5V
- C113 pad 2: +5VA -> +5V
- C114 pad 2: +5VA -> +5V
- C115 pad 2: +5VA -> +5V
- C116 pad 2: +5VA -> +5V
- C117 pad 1: Net-(C117-Pad1) -> +5VA
- C117 pad 2: +5VA -> +5V
- C118 pad 1: Net-(C118-Pad1) -> +5VA
- C118 pad 2: +5VA -> +5V
- C119 pad 1: Net-(C119-Pad1) -> +5VA
- C119 pad 2: +5VA -> +5V
- C12 pad 2: +5VA -> +5V
- C120 pad 1: Net-(C120-Pad1) -> +5VA
- C120 pad 2: +5VA -> +5V
- C121 pad 2: +5VA -> +5V
- C122 pad 1: +5V -> Net-(C122-Pad1)
- C122 pad 2: +5VA -> +5V
- C123 pad 1: TEMP_3 -> Net-(C123-Pad1)
- C123 pad 2: +5VA -> +5V
- C124 pad 1: TEMP_1 -> Net-(C124-Pad1)
- C124 pad 2: +5VA -> +5V
- C125 pad 1: TEMP_2 -> Net-(C125-Pad1)
- C125 pad 2: +5VA -> +5V
- C126 pad 1: Net-(U39-Pad3) -> +5V
- C126 pad 2: +5VA -> +5V
- C127 pad 1: Net-(U40-Pad3) -> TEMP_1
- C127 pad 2: +5VA -> +5V
- C128 pad 1: Net-(U41-Pad3) -> Net-(C128-Pad1)
- C128 pad 2: +5VA -> +5V
- C129 pad 2: +5VA -> +5V
- C13 pad 2: +5VA -> +5V
- C130 pad 2: +5VA -> +5V
- C131 pad 2: +5VA -> +5V
- C132 pad 2: +5VA -> +5V
- C14 pad 2: +5VA -> +5V
- C15 pad 2: +5VA -> +5V
- C16 pad 2: +5VA -> +5V
- C2 pad 2: +5VA -> +5V
- C20 pad 1: MAG_AMP_3 -> MAG_AMP_1
- C20 pad 2: +5VA -> +5V
- C21 pad 1: MAG_AMP_2 -> MAG_LIM_1
- C21 pad 2: +5VA -> +5V
- C22 pad 1: MAG_AMP_1 -> MAG_AMP_2
- C22 pad 2: +5VA -> +5V
- C23 pad 1: MAG_LIM_1 -> MAG_LIM_2
- C23 pad 2: +5VA -> +5V
- C24 pad 1: MAG_LIM_2 -> MAG_AMP_3
- C24 pad 2: +5VA -> +5V
- C25 pad 1: MAG_AMP_3 -> MAG_LIM_3
- C25 pad 2: +5VA -> +5V
- C26 pad 2: +5VA -> +5V
- C27 pad 2: +5VA -> +5V
- C28 pad 2: +5VA -> +5V
- C29 pad 2: +5VA -> +5V
- C3 pad 2: +5VA -> +5V
- C30 pad 2: +5VA -> +5V
- C31 pad 2: +5VA -> +5V
- C32 pad 2: +5VA -> +5V
- C33 pad 2: +5VA -> +5V
- C34 pad 2: +5VA -> +5V
- C35 pad 2: +5VA -> +5V
- C36 pad 2: +5VA -> +5V
- C37 pad 2: +5VA -> +5V
- C38 pad 2: +5VA -> +5V
- C39 pad 2: +5VA -> +5V
- C4 pad 2: +5VA -> +5V
- C40 pad 2: +5VA -> +5V
- C41 pad 2: +5VA -> +5V
- C42 pad 1: +5V -> Net-(C42-Pad1)
- C42 pad 2: +5VA -> +5V
- C43 pad 1: MOT_ENC_2 -> Net-(C43-Pad1)
- C43 pad 2: +5VA -> +5V
- C44 pad 1: MOT_ENC_1 -> Net-(C44-Pad1)
- C44 pad 2: +5VA -> +5V
- C45 pad 1: MAG_LIM_1 -> Net-(C45-Pad1)
- C45 pad 2: +5VA -> +5V
- C46 pad 1: MAG_LIM_2 -> +5V
- C46 pad 2: +5VA -> +5V
- C47 pad 1: MOT_ENC_3 -> MOT_ENC_1
- C47 pad 2: +5VA -> +5V
- C48 pad 1: MAG_LIM_3 -> Net-(C48-Pad1)
- C48 pad 2: +5VA -> +5V
- C49 pad 1: +5V -> MOT_ENC_2
- C49 pad 2: +5VA -> +5V
- C5 pad 2: +5VA -> +5V
- C50 pad 1: +5VA -> Net-(C50-Pad1)
- C50 pad 2: +5VA -> +5V
- C51 pad 1: +5VA -> MOT_ENC_3
- C51 pad 2: +5VA -> +5V
- C52 pad 1: +5VA -> Net-(C52-Pad1)
- C52 pad 2: +5VA -> +5V
- C53 pad 1: +5VA -> +5V
- C53 pad 2: +5VA -> +5V
- C54 pad 2: +5VA -> +5V
- C55 pad 2: +5VA -> +5V
- C56 pad 2: +5VA -> +5V
- C57 pad 2: +5VA -> +5V
- C58 pad 2: +5VA -> +5V
- C59 pad 2: +5VA -> +5V
- C6 pad 2: +5VA -> +5V
- C60 pad 2: +5VA -> +5V
- C61 pad 2: +5VA -> +5V
- C62 pad 1: Net-(C62-Pad1) -> +5VA
- C62 pad 2: +5VA -> +5V
- C63 pad 1: Net-(C63-Pad1) -> +5VA
- C63 pad 2: +5VA -> +5V
- C64 pad 1: Net-(C64-Pad1) -> +5VA
- C64 pad 2: +5VA -> +5V
- C65 pad 1: LC_LIM_1 -> +5VA
- C65 pad 2: +5VA -> +5V
- C66 pad 1: LC_LIM_2 -> Net-(C66-Pad1)
- C66 pad 2: +5VA -> +5V
- C67 pad 1: +5VA -> LC_LIM_1
- C67 pad 2: +5VA -> +5V
- C68 pad 1: +5VA -> Net-(C68-Pad1)
- C68 pad 2: +5VA -> +5V
- C69 pad 1: +5VA -> LC_LIM_2
- C69 pad 2: +5VA -> +5V
- C7 pad 2: +5VA -> +5V
- C70 pad 1: LC_LIM_3 -> Net-(C70-Pad1)
- C70 pad 2: +5VA -> +5V
- C71 pad 2: +5VA -> +5V
- C72 pad 2: +5VA -> +5V
- C73 pad 2: +5VA -> +5V
- C74 pad 2: +5VA -> +5V
- C75 pad 2: +5VA -> +5V
- C76 pad 2: +5VA -> +5V
- C77 pad 1: +5VA -> LC_LIM_3
- C77 pad 2: +5VA -> +5V
- C78 pad 2: +5VA -> +5V
- C79 pad 2: +5VA -> +5V
- C8 pad 2: +5VA -> +5V
- C80 pad 2: +5VA -> +5V
- C81 pad 2: +5VA -> +5V
- C82 pad 2: +5VA -> +5V
- C83 pad 2: +5VA -> +5V
- C84 pad 2: +5VA -> +5V
- C85 pad 2: +5VA -> +5V
- C86 pad 1: TOR_MOT_2 -> +5VA
- C86 pad 2: +5VA -> +5V
- C87 pad 1: LC_LIM_1 -> +5VA
- C87 pad 2: +5VA -> +5V
- C88 pad 1: LC_LIM_2 -> +5VA
- C88 pad 2: +5VA -> +5V
- C89 pad 1: TOR_MOT_3 -> +5VA
- C89 pad 2: +5VA -> +5V
- C9 pad 2: +5VA -> +5V
- C90 pad 2: +5VA -> +5V
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Other:
- board outline removed
- board text removed: "ICSP"
