File: ExoFlexV2/ExoFlex_Kicad.kicad_pcb (KiCad board)
At the start: 2 copper layers, 488 parts, among them J1 24V, J10 AMP_EVE1, J11 SWIVEL, J12 TOR_EXT1, J13 TOR_DOR1, J14 TOR_EVE1, J15 TOR_LIM, J16 AMP_LIM, J17 TOR2, J18 LIMITSWITCH, J19 PROXIMITY, J2 5V, J20 AMP2, J3 24V, J4 CN8, J5 CN9, J6 CN7, J7 CN10, J8 AMP_EXT1, J9 AMP_DOR1, K1 UD2-5NU, U1 PTSM36ADBZR, U10 ADCMP602BRMZ, U11 ADCMP602BRMZ, U12 ADCMP602BRMZ, U13 SN74LVC3G14DCUT_V2, U14 SN74HC7032D_V2, U15 SN74LV4T08PWR_V2, U16 SN74HC7032D_V2, U17 74LV244PW, U18 74LV244PW, U19 SN74LVC3G14DCUT_V2, U2 STPS20M100SG-TR, U20 SN74HC7032D_V2, U21 ADCMP602BRMZ, U22 ADCMP602BRMZ, U23 ADCMP602BRMZ, U24 MCP6001T-I_OT, U25 MCP6001T-I_OT, U26 MCP6001T-I_OT, U27 ADCMP602BRMZ, U28 ADCMP602BRMZ, U29 ADCMP602BRMZ, U3 CD4044BPWR, U30 ADCMP602BRMZ, U31 ADCMP602BRMZ, U32 ADCMP602BRMZ, U33 SN74LVC3G14DCUT_V2, U34 SN74LV4T08PWR_V2, U35 SN74HC7032D_V2, U36 ADCMP602BRMZ, U37 ADCMP602BRMZ, U38 ADCMP602BRMZ, U4 LMZ23603TZ_NOPB, U5 TPS7A4701RGWR, U6 SN74HC7032D_V2, U7 SN74HC7032D_V2, U8 SN74LV4T08PWR_V2, U9 SN74LV4T08PWR_V2

Commit message: Placement encore
Parts:
- added C133: 0,01uF, Capacitor_SMD:C_0603_1608Metric, F.Cu at (119.8, 285.9)
- added R95: 7,5k, Resistor_SMD:R_0603_1608Metric, F.Cu at (150.5, 122.6)
- added TP131: 5005, FootPrint:KEYSTONE_5005, F.Cu at (142.4, 120.1)
- C1: value 150uF 50V -> 10uF; footprint FootPrint:CAP_EEHZS1H151P -> Capacitor_SMD:C_0603_1608Metric
- C10, C17: value 1uF -> 10uF
- C105: value 0,1uF -> 0,01uF
- C106, C113, C33, C54: value 0,01uF -> 0,1uF
- C109, C66, C90: value 1nF -> 0,01uF
- C11: value 47uF -> 1uF; footprint Capacitor_SMD:C_1206_3216Metric -> Capacitor_SMD:C_0603_1608Metric
- C110: value 10 uF -> 1nF
- C111, C122, C123, C124, C125, C40, C41, C42, C43, C44, C45: value 10 uF -> 10uF
- C112, C126, C46: value 0,1uF -> 10uF
- C12: value 10uF -> 47uF; footprint Capacitor_SMD:C_0603_1608Metric -> Capacitor_SMD:C_1206_3216Metric
- C121: value 10 uF -> 0,01uF
- C127, C47: value 1nF -> 0,1uF
- C129, C26, C78, C96: value 0,01uF -> 1nF
- C2: value 10 uF -> 150uF 50V; footprint Capacitor_SMD:C_0805_2012Metric -> FootPrint:CAP_EEHZS1H151P
- C20: value 1nF -> 1uF
- C27, C28, C29, C30, C31, C34, C35, C36, C37, C38: moved to B.Cu
- C3: value 0,047uF -> 10 uF; footprint Capacitor_SMD:C_0603_1608Metric -> Capacitor_SMD:C_0805_2012Metric
- C32: value 0,1uF -> 0,01uF; moved to B.Cu
- C39: value 10 uF -> 0,01uF; moved to B.Cu
- C4: value 100uF 20V -> 0,047uF; footprint FootPrint:CAP_PC_8X7_NCH -> Capacitor_SMD:C_0603_1608Metric
- C5: value 220uF 50V -> 100uF 20V; footprint FootPrint:CAP_EEHZS1H221P -> FootPrint:CAP_PC_8X7_NCH
- C53: value 0,1uF -> 1nF
- C6: value 0,047uF -> 220uF 50V; footprint Capacitor_SMD:C_0603_1608Metric -> FootPrint:CAP_EEHZS1H221P
- C7: value 100uF -> 0,047uF; footprint Capacitor_SMD:C_1210_3225Metric -> Capacitor_SMD:C_0603_1608Metric
- C71: value 0,1uF -> 1nF; moved to F.Cu
- C74: value 1uF -> 0,1uF
- C77: value 1nF -> 1uF; moved to B.Cu
- C8: value 220uF 20V -> 100uF; footprint FootPrint:CAP_20SVPK220M -> Capacitor_SMD:C_1210_3225Metric
- C9: value 10uF -> 220uF 20V; footprint Capacitor_SMD:C_0603_1608Metric -> FootPrint:CAP_20SVPK220M
- R1: value 1,5k -> 5k
- R12: value 150 -> 5k
- R13: value 3,6k -> 150
- R14: value 2,5k -> 3,6k
- R15: value 7,5k -> 2,5k
- R2: value 1,1k -> 1,5k
- R21, R73: value 5k -> 7,5k
- R28, R90: value 0Ω -> 5k
- R3: value 6,8k -> 1,1k
- R31, R41, R44, R67, R91: value 7,5k -> 0Ω
- R37, R42, R76: value 0Ω -> 7,5k
- R4: value RE1C002UNTCL -> 6,8k; footprint FootPrint:DIO_RB558WMF_ROM -> Resistor_SMD:R_0603_1608Metric
- R48: value 10k -> 7,5k
- R5: value 23,7 -> RE1C002UNTCL; footprint Resistor_SMD:R_0603_1608Metric -> FootPrint:DIO_RB558WMF_ROM
- R51: value 220k -> 10k
- R54: value 2M -> 220k
- R57: value 430k -> 2M
- R6: value 25,5k 1% -> 23,7
- R60: value 7,5k -> 430k
- R61: value 2M -> 7,5k
- R64: value 0Ω -> 2M
- R7: value 10k -> 25,5k 1%
- R75: value 7,5k -> 5k
- R8: value 2,5k -> 10k
- R85: value 5k -> 0Ω
- R9: value 5k -> 2,5k
- R92: value 0 ohm -> 7,5k
- R94: value 7,5k -> 0 ohm
- U10: value ADCMP602BRMZ -> SN74LV4T08PWR_V2; footprint FootPrint:ADCMP602BRMZ -> FootPrint:SN74LV4T08PWR
- U13: value SN74LVC3G14DCUT_V2 -> ADCMP602BRMZ; footprint FootPrint:SN74LVC3G14DCUT -> FootPrint:ADCMP602BRMZ
- U14: value SN74HC7032D_V2 -> SN74LVC3G14DCUT_V2; footprint FootPrint:SN74HC7032D -> FootPrint:SN74LVC3G14DCUT
- U15, U8: value SN74LV4T08PWR_V2 -> SN74HC7032D_V2; footprint FootPrint:SN74LV4T08PWR -> FootPrint:SN74HC7032D
- U16: value SN74HC7032D_V2 -> SN74LV4T08PWR_V2; footprint FootPrint:SN74HC7032D -> FootPrint:SN74LV4T08PWR
- U17: value 74LV244PW -> SN74HC7032D_V2; footprint FootPrint:DB20 -> FootPrint:SN74HC7032D
- U3: value CD4044BPWR -> 74LV244PW; footprint FootPrint:CD4044BPWR -> FootPrint:DB20
- U4: value LMZ23603TZ_NOPB -> CD4044BPWR; footprint FootPrint:LMZ23603 -> FootPrint:CD4044BPWR
- U5: value TPS7A4701RGWR -> LMZ23603TZ_NOPB; footprint FootPrint:TPS7A470 -> FootPrint:LMZ23603
- U6: value SN74HC7032D_V2 -> TPS7A4701RGWR; footprint FootPrint:SN74HC7032D -> FootPrint:TPS7A470
- moved C2 271.3 mm to (116.8, 54.1)
- moved C9 259.8 mm to (133.0, 64.0)
- moved C6 255.5 mm to (117.5, 38.6)
- moved C34 254.4 mm to (66.7, 76.9), turned to 180 degrees
- moved R6 250.5 mm to (284.0, 149.5)
- moved R4 250.5 mm to (284.0, 146.9)
- moved R3 250.5 mm to (293.0, 141.1)
- moved R5 250.5 mm to (288.0, 146.9)
- moved R7 250.5 mm to (288.0, 141.3)
- moved R2 250.5 mm to (293.0, 138.6)
- moved U37 242.5 mm to (73.1, 292.0)
- moved U6 242.5 mm to (58.6, 280.3)
- moved C53 236.6 mm to (57.3, 100.0)
- moved C32 235.0 mm to (73.1, 95.9)
- moved D1 234.3 mm to (272.3, 131.2)
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Connections:
- C1 pad 1: +24V -> Net-(C1-Pad1)
- C10 pad 1: Net-(C10-Pad1) -> Net-(C7-Pad1)
- C105 pad 1: +5V -> +5VA
- C106 pad 1: +5VA -> +5V
- C109 pad 1: MAG_AMP_4 -> +5VA
- C11 pad 1: +5VA -> Net-(C11-Pad1)
- C110 pad 1: Net-(C110-Pad1) -> MAG_AMP_4
- C112 pad 1: +5V -> Net-(C112-Pad1)
- C113 pad 1: +5VA -> +5V
- C121 pad 1: Net-(C121-Pad1) -> +5VA
- C126 pad 1: +5V -> Net-(C126-Pad1)
- C127 pad 1: TEMP_1 -> +5V
- C128 pad 1: Net-(C128-Pad1) -> TEMP_1
- C129 pad 1: +5VA -> Net-(C129-Pad1)
- C17 pad 1: +5V -> +5VA
- C20 pad 1: MAG_AMP_1 -> +5V
- C21 pad 1: MAG_LIM_1 -> MAG_AMP_1
- C22 pad 1: MAG_AMP_2 -> MAG_LIM_1
- C23 pad 1: MAG_LIM_2 -> MAG_AMP_2
- C24 pad 1: MAG_AMP_3 -> MAG_LIM_2
- C25 pad 1: MAG_LIM_3 -> MAG_AMP_3
- C26 pad 1: +5VA -> MAG_LIM_3
- C32 pad 1: +5V -> +5VA
- C33 pad 1: +5VA -> +5V
- C39 pad 1: Net-(C39-Pad1) -> +5VA
- C4 pad 1: +5V -> +24V
- C46 pad 1: +5V -> Net-(C46-Pad1)
- C47 pad 1: MOT_ENC_1 -> +5V
- C48 pad 1: Net-(C48-Pad1) -> MOT_ENC_1
- C49 pad 1: MOT_ENC_2 -> Net-(C49-Pad1)
- C5 pad 1: +24V -> +5V
- C50 pad 1: Net-(C50-Pad1) -> MOT_ENC_2
- C51 pad 1: MOT_ENC_3 -> Net-(C51-Pad1)
- C52 pad 1: Net-(C52-Pad1) -> MOT_ENC_3
- C53 pad 1: +5V -> Net-(C53-Pad1)
- C54 pad 1: +5VA -> +5V
- C6 pad 1: Net-(C6-Pad1) -> +24V
- C66 pad 1: Net-(C66-Pad1) -> +5VA
- C67 pad 1: LC_LIM_1 -> Net-(C67-Pad1)
- C68 pad 1: Net-(C68-Pad1) -> LC_LIM_1
- C69 pad 1: LC_LIM_2 -> Net-(C69-Pad1)
- C7 pad 1: Net-(C6-Pad1) -> Net-(C7-Pad1)
- C70 pad 1: Net-(C70-Pad1) -> LC_LIM_2
- C71 pad 1: +5VA -> Net-(C71-Pad1)
- C77 pad 1: LC_LIM_3 -> +5VA
- C78 pad 1: +5VA -> LC_LIM_3
- C8 pad 1: Net-(C6-Pad1) -> Net-(C7-Pad1)
- C9 pad 1: Net-(C6-Pad1) -> Net-(C7-Pad1)
- C90 pad 1: TOR_MOT_1 -> +5VA
- C91 pad 1: Net-(C91-Pad1) -> TOR_MOT_1
- C92 pad 1: TOR_MOT_2 -> Net-(C92-Pad1)
- C93 pad 1: Net-(C93-Pad1) -> TOR_MOT_2
- C94 pad 1: TOR_MOT_3 -> Net-(C94-Pad1)
- C95 pad 1: Net-(C95-Pad1) -> TOR_MOT_3
- C96 pad 1: +5VA -> Net-(C96-Pad1)
- R1 pad 1: +5V -> RESET
- R1 pad 2: Net-(R1-Pad2) -> Net-(C1-Pad1)
- R10 pad 1: +5VA -> +5V
- R10 pad 2: MAG1_POT1 -> MAG2_POT2
- R11 pad 1: +5V -> +5VA
- R11 pad 2: MAG1_POT2 -> MAG1_POT1
- R12 pad 1: +5VA -> +5V
- R12 pad 2: Net-(R12-Pad2) -> MAG1_POT2
- R13 pad 1: Net-(R12-Pad2) -> +5VA
- R13 pad 2: MAG3_POT1 -> Net-(R13-Pad2)
- R14 pad 1: +5V -> Net-(R13-Pad2)
- R14 pad 2: MAG3_POT2 -> MAG3_POT1
- R15 pad 1: MAG_OUT_1 -> +5V
- R15 pad 2: MAG_AMP_1 -> MAG3_POT2
- R16 pad 1: MAG1_POT_OUT -> MAG_OUT_1
- R16 pad 2: MAG_LIM_1 -> MAG_AMP_1
- R17 pad 1: MAG_OUT_2 -> MAG1_POT_OUT
- R17 pad 2: MAG_AMP_2 -> MAG_LIM_1
- R18 pad 1: MAG2_POT_OUT -> MAG_OUT_2
- R18 pad 2: MAG_LIM_2 -> MAG_AMP_2
- R19 pad 1: MAG_OUT_3 -> MAG2_POT_OUT
- R19 pad 2: MAG_AMP_3 -> MAG_LIM_2
- R20 pad 1: MAG3_POT_OUT -> MAG_OUT_3
- R20 pad 2: MAG_LIM_3 -> MAG_AMP_3
- R21 pad 1: MAX_SW_1 -> MAG3_POT_OUT
- R21 pad 2: Net-(C39-Pad1) -> MAG_LIM_3
- R22 pad 1: MAX_SW_2 -> MAX_SW_1
- R23 pad 1: MAX_SW_3 -> MAX_SW_2
- R24 pad 1: MIN_SW_1 -> MAX_SW_3
- R25 pad 1: MIN_SW_2 -> MIN_SW_1
- R26 pad 1: MIN_SW_3 -> MIN_SW_2
- R27 pad 1: URG_USER_1 -> MIN_SW_3
- R28 pad 1: Net-(R28-Pad1) -> URG_USER_1
- R28 pad 2: MOT_ENC_OUT_1 -> Net-(C46-Pad1)
- R29 pad 2: MOT_ENC_OUT_2 -> MOT_ENC_OUT_1
- R3 pad 1: Net-(R2-Pad2) -> +5V
- R30 pad 2: MOT_ENC_OUT_3 -> MOT_ENC_OUT_2
- R31 pad 1: MOT_ENC_OUT_1 -> Net-(R31-Pad1)
- R31 pad 2: MOT_ENC_1 -> MOT_ENC_OUT_3
- R32 pad 1: MAG1_POT_OUT -> MOT_ENC_OUT_1
- R32 pad 2: Net-(C48-Pad1) -> MOT_ENC_1
- R33 pad 1: MOT_ENC_OUT_2 -> MAG1_POT_OUT
- R33 pad 2: MOT_ENC_2 -> Net-(C49-Pad1)
- R34 pad 1: MAG2_POT_OUT -> MOT_ENC_OUT_2
- R34 pad 2: Net-(C50-Pad1) -> MOT_ENC_2
- R35 pad 1: MOT_ENC_OUT_3 -> MAG2_POT_OUT
- R35 pad 2: MOT_ENC_3 -> Net-(C51-Pad1)
- R36 pad 1: MAG3_POT_OUT -> MOT_ENC_OUT_3
- R36 pad 2: Net-(C52-Pad1) -> MOT_ENC_3
- R37 pad 1: +5VA -> MAG3_POT_OUT
- R37 pad 2: LC1_POT1 -> Net-(C53-Pad1)
- R38 pad 1: +5V -> +5VA
- R38 pad 2: LC1_POT2 -> LC1_POT1
- R39 pad 1: +5VA -> +5V
- R39 pad 2: LC2_POT1 -> LC1_POT2
- R4 pad 1: /POWER/LATCH_Q1 -> Net-(R3-Pad2)
- R4 pad 2: +5V -> Net-(R4-Pad2)
- R40 pad 1: +5V -> +5VA
- R40 pad 2: LC2_POT2 -> LC2_POT1
- R41 pad 1: LC2_POT_OUT -> +5V
- R41 pad 2: LC_LIM_2 -> LC2_POT2
- R42 pad 1: +5VA -> LC2_POT_OUT
- R42 pad 2: LC3_POT1 -> LC_LIM_2
- R43 pad 1: +5V -> +5VA
- R43 pad 2: LC3_POT2 -> LC3_POT1
- R44 pad 1: LC1_POT_OUT -> +5V
- R44 pad 2: LC_LIM_1 -> LC3_POT2
- R45 pad 1: LC_O+_2 -> LC1_POT_OUT
- R45 pad 2: Net-(C68-Pad1) -> LC_LIM_1
- R46 pad 1: LC_O+_1 -> LC_O+_2
- R46 pad 2: Net-(C66-Pad1) -> Net-(C69-Pad1)
- R47 pad 1: LC_O+_3 -> LC_O+_1
- R47 pad 2: Net-(C70-Pad1) -> Net-(C67-Pad1)
- R48 pad 1: +5V -> LC_O+_3
- R48 pad 2: Net-(R48-Pad2) -> Net-(C71-Pad1)
- R5 pad 1: Net-(R3-Pad2) -> /POWER/LATCH_Q1
- R5 pad 2: Net-(C6-Pad1) -> +5V
- R51 pad 1: Net-(R48-Pad2) -> +5V
- R54 pad 1: Net-(R48-Pad2) -> Net-(R51-Pad2)
- R57 pad 2: Net-(R54-Pad2) -> Net-(R57-Pad2)
- R6 pad 1: +5V -> Net-(R4-Pad2)
- R6 pad 2: Net-(R6-Pad2) -> Net-(C7-Pad1)
- R60 pad 1: LC3_POT_OUT -> Net-(R54-Pad2)
- R60 pad 2: LC_LIM_3 -> Net-(R57-Pad2)
- R61 pad 1: Net-(R54-Pad2) -> LC3_POT_OUT
- R61 pad 2: LC_TOR_1 -> LC_LIM_3
- R62 pad 2: LC_TOR_2 -> LC_TOR_1
- R63 pad 2: LC_TOR_3 -> LC_TOR_2
- R64 pad 1: Net-(R64-Pad1) -> Net-(R57-Pad2)
- R64 pad 2: TOR_MOT_OUT_1 -> LC_TOR_3
- R65 pad 2: TOR_MOT_OUT_2 -> TOR_MOT_OUT_1
- R66 pad 2: TOR_MOT_OUT_3 -> TOR_MOT_OUT_2
- R67 pad 1: TOR_MOT_OUT_1 -> Net-(R67-Pad1)
- R67 pad 2: TOR_MOT_1 -> TOR_MOT_OUT_3
- R68 pad 1: LC1_POT_OUT -> TOR_MOT_OUT_1
- R68 pad 2: Net-(C91-Pad1) -> TOR_MOT_1
- R69 pad 1: TOR_MOT_OUT_2 -> LC1_POT_OUT
- R69 pad 2: TOR_MOT_2 -> Net-(C92-Pad1)
- R7 pad 1: +5VA -> +5V
- R7 pad 2: Net-(R6-Pad2) -> Net-(R7-Pad2)
- R70 pad 1: LC2_POT_OUT -> TOR_MOT_OUT_2
- R70 pad 2: Net-(C93-Pad1) -> TOR_MOT_2
- R71 pad 1: TOR_MOT_OUT_3 -> LC2_POT_OUT
- R71 pad 2: TOR_MOT_3 -> Net-(C94-Pad1)
- R72 pad 1: LC3_POT_OUT -> TOR_MOT_OUT_3
- R72 pad 2: Net-(C95-Pad1) -> TOR_MOT_3
- R73 pad 1: MAX_SW_4 -> LC3_POT_OUT
- R73 pad 2: Net-(C110-Pad1) -> Net-(C96-Pad1)
- R74 pad 1: MAX_SW_5 -> MAX_SW_4
- R75 pad 1: MAG_OUT_4 -> MAX_SW_5
- R75 pad 2: MAG_AMP_4 -> Net-(C112-Pad1)
- R76 pad 1: Net-(R76-Pad1) -> MAG_OUT_4
- R76 pad 2: +5VA -> MAG_AMP_4
- R77 pad 1: +5V -> Net-(R77-Pad1)
- R77 pad 2: Net-(R76-Pad1) -> +5VA
- R78 pad 1: Net-(R78-Pad1) -> +5V
- R78 pad 2: +5VA -> Net-(R77-Pad1)
- R79 pad 1: +5V -> Net-(R79-Pad1)
- R79 pad 2: Net-(R78-Pad1) -> +5VA
- R8 pad 2: MAG2_POT1 -> Net-(R7-Pad2)
- R80 pad 1: Net-(R80-Pad1) -> +5V
- R80 pad 2: PROX_OUT_1 -> Net-(R79-Pad1)
- R81 pad 2: PROX_OUT_2 -> PROX_OUT_1
- R82 pad 2: PROX_OUT_3 -> PROX_OUT_2
- R83 pad 2: BUT_PROX_1 -> PROX_OUT_3
- R84 pad 2: BUT_PROX_2 -> BUT_PROX_1
- R85 pad 1: PROX_OUT_1 -> Net-(R85-Pad1)
- R85 pad 2: Net-(C121-Pad1) -> BUT_PROX_2
- R86 pad 1: PROX_OUT_2 -> PROX_OUT_1
- R87 pad 1: PROX_OUT_3 -> PROX_OUT_2
- R88 pad 1: BUT_PROX_1 -> PROX_OUT_3
- R89 pad 1: BUT_PROX_2 -> BUT_PROX_1
- R9 pad 1: +5V -> +5VA
- R9 pad 2: MAG2_POT2 -> MAG2_POT1
- R90 pad 1: Net-(R90-Pad1) -> BUT_PROX_2
- R90 pad 2: TEMP_OUT_1 -> Net-(C126-Pad1)
- R91 pad 1: TEMP_OUT_1 -> Net-(R91-Pad1)
- R91 pad 2: TEMP_1 -> TEMP_OUT_1
- R92 pad 1: +5VA -> TEMP_OUT_1
- R92 pad 2: Net-(R92-Pad2) -> TEMP_1
- R93 pad 1: +5V -> +5VA
- R93 pad 2: Net-(R92-Pad2) -> Net-(R93-Pad2)
- R94 pad 1: Net-(R92-Pad2) -> +5V
- R94 pad 2: Net-(C128-Pad1) -> Net-(R93-Pad2)
- TP103 pad TP: Net-(R80-Pad1) -> Net-(R81-Pad1)
- TP104 pad TP: Net-(R81-Pad1) -> Net-(R82-Pad1)
- TP105 pad TP: Net-(R82-Pad1) -> Net-(R83-Pad1)
- TP106 pad TP: Net-(R83-Pad1) -> Net-(R84-Pad1)
- TP107 pad TP: Net-(R84-Pad1) -> Net-(R85-Pad1)
- TP118 pad TP: Net-(R90-Pad1) -> Net-(R91-Pad1)
- TP2 pad TP: RESET -> Net-(TP2-PadTP)
- TP44 pad TP: Net-(R28-Pad1) -> Net-(R29-Pad1)
- TP45 pad TP: Net-(R29-Pad1) -> Net-(R30-Pad1)
- TP46 pad TP: Net-(R30-Pad1) -> Net-(R31-Pad1)
- TP48 pad TP: Net-(C48-Pad1) -> Net-(C49-Pad1)
- TP50 pad TP: Net-(C50-Pad1) -> Net-(C51-Pad1)
- TP52 pad TP: Net-(C52-Pad1) -> Net-(C53-Pad1)
- TP7 pad TP: Net-(C6-Pad1) -> Net-(C7-Pad1)
- TP73 pad TP: Net-(R64-Pad1) -> Net-(R65-Pad1)
- TP74 pad TP: Net-(R65-Pad1) -> Net-(R66-Pad1)
- TP75 pad TP: Net-(R66-Pad1) -> Net-(R67-Pad1)
- TP77 pad TP: Net-(C91-Pad1) -> Net-(C92-Pad1)
- TP79 pad TP: Net-(C93-Pad1) -> Net-(C94-Pad1)
- TP81 pad TP: Net-(C95-Pad1) -> Net-(C96-Pad1)
- TP89 pad TP: Net-(R76-Pad1) -> Net-(R77-Pad1)
- TP90 pad TP: Net-(R78-Pad1) -> Net-(R79-Pad1)
- U10 pad 1: +5VA -> Net-(TP14-PadTP)
- U10 pad 2: MAG_AMP_1 -> LEFTRIGHT_SEC
- U10 pad 3: MAG_LIM_1 -> Net-(TP18-PadTP)
- U10 pad 4: unconnected-(U10-Pad4) -> (no net)
- U10 pad 5: unconnected-(U10-Pad5) -> (no net)
- U10 pad 6: +5V -> (no net)
- U10 pad 7: Net-(TP26-PadTP) -> +5V
- U10 pad 8: +5VA -> Net-(TP100-PadTP)
- U11 pad 2: MAG_AMP_2 -> MAG_AMP_1
- U11 pad 3: MAG_LIM_2 -> MAG_LIM_1
- U11 pad 7: Net-(TP27-PadTP) -> Net-(TP26-PadTP)
- U12 pad 2: MAG_AMP_3 -> MAG_AMP_2
- U12 pad 3: MAG_LIM_3 -> MAG_LIM_2
- U12 pad 7: Net-(TP28-PadTP) -> Net-(TP27-PadTP)
- U13 pad 1: Net-(TP53-PadTP) -> +5VA
- U13 pad 2: Net-(TP69-PadTP) -> MAG_AMP_3
- U13 pad 3: Net-(TP27-PadTP) -> MAG_LIM_3
- U13 pad 4: (no net) -> unconnected-(U13-Pad4)
- U13 pad 5: Net-(TP29-PadTP) -> unconnected-(U13-Pad5)
- U13 pad 6: Net-(TP66-PadTP) -> +5V
- U13 pad 7: +5V -> Net-(TP28-PadTP)
- U13 pad 8: +5V -> +5VA
- U14 pad 1: (no net) -> Net-(TP53-PadTP)
- U14 pad 2: (no net) -> Net-(TP69-PadTP)
- U14 pad 3: (no net) -> Net-(TP27-PadTP)
- U14 pad 4: Net-(TP55-PadTP) -> (no net)
- U14 pad 5: Net-(TP53-PadTP) -> Net-(TP29-PadTP)
- U14 pad 6: Net-(TP57-PadTP) -> Net-(TP66-PadTP)
- U14 pad 7: (no net) -> +5V
- U14 pad 8: MOT_ENC_SEC -> +5V
- U15 pad 1: Net-(TP56-PadTP) -> (no net)
- U15 pad 10: Net-(TP68-PadTP) -> Net-(TP58-PadTP)
- U15 pad 11: Net-(TP42-PadTP) -> Net-(TP30-PadTP)
- U15 pad 12: Net-(TP40-PadTP) -> Net-(TP26-PadTP)
- U15 pad 13: SWMAX3 -> Net-(TP27-PadTP)
- U15 pad 14: +5V -> (no net)
- U15 pad 2: Net-(TP54-PadTP) -> (no net)
- U15 pad 3: Net-(TP58-PadTP) -> (no net)
- U15 pad 4: Net-(TP29-PadTP) -> Net-(TP55-PadTP)
- U15 pad 5: Net-(TP28-PadTP) -> Net-(TP53-PadTP)
- U15 pad 6: Net-(TP31-PadTP) -> Net-(TP57-PadTP)
- U15 pad 7: +5V -> (no net)
- U15 pad 8: Net-(TP71-PadTP) -> MOT_ENC_SEC
- U15 pad 9: Net-(TP69-PadTP) -> Net-(TP57-PadTP)
- U16 pad 1: Net-(TP30-PadTP) -> Net-(TP56-PadTP)
- U16 pad 10: Net-(TP71-PadTP) -> Net-(TP68-PadTP)
- U16 pad 11: Net-(TP41-PadTP) -> Net-(TP42-PadTP)
- U16 pad 12: SWMAX1 -> Net-(TP40-PadTP)
- U16 pad 13: SWMAX2 -> SWMAX3
- U16 pad 2: Net-(TP31-PadTP) -> Net-(TP54-PadTP)
- U16 pad 3: MAG_AMP_SEC -> Net-(TP58-PadTP)
- U16 pad 4: Net-(TP67-PadTP) -> Net-(TP29-PadTP)
- U16 pad 5: Net-(TP66-PadTP) -> Net-(TP28-PadTP)
- U16 pad 6: Net-(TP70-PadTP) -> Net-(TP31-PadTP)
- U16 pad 8: LC_TOR_SEC -> Net-(TP71-PadTP)
- U16 pad 9: Net-(TP70-PadTP) -> Net-(TP69-PadTP)
- U17 pad 1: +5V -> Net-(TP30-PadTP)
- U17 pad 10: +5V -> Net-(TP71-PadTP)
- U17 pad 11: Net-(C123-Pad1) -> Net-(TP41-PadTP)
- U17 pad 12: SWMAX4 -> SWMAX1
- U17 pad 13: Net-(C122-Pad1) -> SWMAX2
- U17 pad 14: SWMAX3 -> +5V
- U17 pad 2: Net-(C39-Pad1) -> Net-(TP31-PadTP)
- U17 pad 3: SWMAX5 -> MAG_AMP_SEC
- U17 pad 4: Net-(C40-Pad1) -> Net-(TP67-PadTP)
- U17 pad 5: PROX_1 -> Net-(TP66-PadTP)
- U17 pad 6: Net-(C41-Pad1) -> Net-(TP70-PadTP)
- U17 pad 7: PROX_2 -> +5V
- U17 pad 8: Net-(C110-Pad1) -> LC_TOR_SEC
- U17 pad 9: PROX_3 -> Net-(TP70-PadTP)
- U18 pad 11: (no net) -> Net-(C112-Pad1)
- U18 pad 12: SWMIN1 -> SWMIN2
- U18 pad 13: Net-(C45-Pad1) -> Net-(C111-Pad1)
- U18 pad 14: (no net) -> SWMAX2
- U18 pad 15: Net-(C44-Pad1) -> Net-(C45-Pad1)
- U18 pad 16: PROX_5 -> SWMIN1
- U18 pad 17: Net-(C43-Pad1) -> Net-(C42-Pad1)
- U18 pad 18: PROX_4 -> SWMAX1
- U18 pad 2: Net-(C124-Pad1) -> Net-(C40-Pad1)
- U18 pad 3: SWMIN2 -> SWMAX3
- U18 pad 4: Net-(C125-Pad1) -> Net-(C43-Pad1)
- U18 pad 6: (no net) -> Net-(C41-Pad1)
- U18 pad 7: URG_SEC -> SWMAX4
- U18 pad 8: Net-(C42-Pad1) -> Net-(C44-Pad1)
- U18 pad 9: (no net) -> SWMAX5
- U21 pad 3: Net-(C48-Pad1) -> Net-(C49-Pad1)
- U22 pad 3: Net-(C50-Pad1) -> Net-(C51-Pad1)
- U23 pad 3: Net-(C52-Pad1) -> Net-(C53-Pad1)
- U24 pad 3: Net-(C66-Pad1) -> Net-(C67-Pad1)
- U24 pad 4: Net-(R48-Pad2) -> Net-(R49-Pad2)
- U25 pad 3: Net-(C68-Pad1) -> Net-(C69-Pad1)
- U25 pad 4: Net-(R49-Pad2) -> Net-(R50-Pad2)
- U26 pad 3: Net-(C70-Pad1) -> Net-(C71-Pad1)
- U26 pad 4: Net-(R50-Pad2) -> Net-(R51-Pad2)
- U3 pad 1: unconnected-(U3-Pad1) -> +5V
- U3 pad 10: unconnected-(U3-Pad10) -> +5V
- U3 pad 11: unconnected-(U3-Pad11) -> (no net)
- U3 pad 12: unconnected-(U3-Pad12) -> PROX_5
- U3 pad 13: /POWER/LATCH_Q1 -> Net-(C124-Pad1)
- U3 pad 14: unconnected-(U3-Pad14) -> PROX_4
- U3 pad 15: unconnected-(U3-Pad15) -> Net-(C123-Pad1)
- U3 pad 16: +5V -> Net-(TP2-PadTP)
- U3 pad 2: unconnected-(U3-Pad2) -> Net-(C46-Pad1)
- U3 pad 3: ALIM_SEC -> PROX_1
- U3 pad 4: RESET -> Net-(C1-Pad1)
- U3 pad 5: +5V -> PROX_2
- U3 pad 6: unconnected-(U3-Pad6) -> Net-(C125-Pad1)
- U3 pad 7: unconnected-(U3-Pad7) -> PROX_3
- U3 pad 8: +5V -> Net-(C126-Pad1)
- U3 pad 9: unconnected-(U3-Pad9) -> (no net)
- U30 pad 3: Net-(C91-Pad1) -> Net-(C92-Pad1)
- U31 pad 3: Net-(C93-Pad1) -> Net-(C94-Pad1)
- U32 pad 3: Net-(C95-Pad1) -> Net-(C96-Pad1)
- U36 pad 3: Net-(R76-Pad1) -> Net-(R77-Pad1)
- U37 pad 2: Net-(R78-Pad1) -> Net-(R79-Pad1)
- U38 pad 3: Net-(C128-Pad1) -> Net-(C129-Pad1)
- U4 pad 1: +24V -> unconnected-(U4-Pad1)
- U4 pad 2: Net-(R1-Pad2) -> unconnected-(U4-Pad2)
- U4 pad 3: unconnected-(U4-Pad3) -> ALIM_SEC
- U4 pad 4: +5V -> Net-(TP2-PadTP)
- U4 pad 5: Net-(R2-Pad2) -> +5V
- U4 pad 7: Net-(C6-Pad1) -> unconnected-(U4-Pad7)
- U4 pad 8: unconnected-(U4-Pad8) -> +5V
- U5 pad 1: +5VA -> +24V
- U5 pad 2: unconnected-(U5-Pad2) -> Net-(R2-Pad2)
- U5 pad 3: Net-(R6-Pad2) -> unconnected-(U5-Pad3)
- U5 pad 4: unconnected-(U5-Pad4) -> +5V
- U5 pad 5: unconnected-(U5-Pad5) -> Net-(R3-Pad2)
- U5 pad 7: +5V -> Net-(C7-Pad1)
- U6 pad 1: Net-(TP19-PadTP) -> +5VA
- U6 pad 10: SW-SEC -> unconnected-(U6-Pad10)
- U6 pad 11: Net-(TP11-PadTP) -> unconnected-(U6-Pad11)
- U6 pad 12: URG_SEC -> unconnected-(U6-Pad12)
- U6 pad 13: TEMP_SEC -> Net-(C7-Pad1)
- U6 pad 14: +5V -> Net-(C11-Pad1)
- U6 pad 2: Net-(TP11-PadTP) -> unconnected-(U6-Pad2)
- U6 pad 3: ALIM_SEC -> Net-(R7-Pad2)
- U6 pad 4: MOT_ENC_SEC -> unconnected-(U6-Pad4)
- U6 pad 5: MAG_AMP_SEC -> unconnected-(U6-Pad5)
- U6 pad 6: Net-(TP10-PadTP) -> unconnected-(U6-Pad6)
- U6 pad 8: Net-(TP12-PadTP) -> unconnected-(U6-Pad8)
- U6 pad 9: Net-(TP10-PadTP) -> unconnected-(U6-Pad9)
- U7 pad 1: LC_TOR_SEC -> Net-(TP19-PadTP)
- U7 pad 10: Net-(TP18-PadTP) -> SW-SEC
- U7 pad 11: Net-(TP14-PadTP) -> Net-(TP11-PadTP)
- U7 pad 12: PROX_SEC -> URG_SEC
- U7 pad 13: BUT_PROX_SEC -> TEMP_SEC
- U7 pad 2: TOR_MOT_SEC -> Net-(TP11-PadTP)
- U7 pad 3: Net-(TP13-PadTP) -> ALIM_SEC
- U7 pad 4: Net-(TP15-PadTP) -> MOT_ENC_SEC
- U7 pad 5: Net-(TP16-PadTP) -> MAG_AMP_SEC
- U7 pad 6: Net-(TP17-PadTP) -> Net-(TP10-PadTP)
- U7 pad 8: Net-(TP19-PadTP) -> Net-(TP12-PadTP)
- U7 pad 9: Net-(TP17-PadTP) -> Net-(TP10-PadTP)
- U8 pad 1: PROX_4 -> LC_TOR_SEC
- U8 pad 10: Net-(TP14-PadTP) -> Net-(TP18-PadTP)
- U8 pad 11: Net-(TP16-PadTP) -> Net-(TP14-PadTP)
- U8 pad 12: Net-(TP14-PadTP) -> PROX_SEC
- U8 pad 13: Net-(TP13-PadTP) -> BUT_PROX_SEC
- U8 pad 2: PROX_5 -> TOR_MOT_SEC
- U8 pad 3: BUT_PROX_SEC -> Net-(TP13-PadTP)
- U8 pad 4: (no net) -> Net-(TP15-PadTP)
- U8 pad 5: (no net) -> Net-(TP16-PadTP)
- U8 pad 6: (no net) -> Net-(TP17-PadTP)
- U8 pad 8: Net-(TP15-PadTP) -> Net-(TP19-PadTP)
- U8 pad 9: Net-(TP12-PadTP) -> Net-(TP17-PadTP)
- U9 pad 1: Net-(TP14-PadTP) -> PROX_4
- U9 pad 10: Net-(TP96-PadTP) -> Net-(TP14-PadTP)
- U9 pad 11: (no net) -> Net-(TP16-PadTP)
- U9 pad 12: (no net) -> Net-(TP14-PadTP)
- U9 pad 13: (no net) -> Net-(TP13-PadTP)
- U9 pad 2: LEFTRIGHT_SEC -> PROX_5
- U9 pad 3: Net-(TP18-PadTP) -> BUT_PROX_SEC
- U9 pad 8: Net-(TP100-PadTP) -> Net-(TP15-PadTP)
- U9 pad 9: Net-(TP95-PadTP) -> Net-(TP12-PadTP)

Commit message: Placement done V1
Parts:
- C100, C101, C102, C103, C104, C105, C106, C107, C108, C109, C113, C114, C115, C116, C117, C118, C119, C120, C121, C127, C130, C131, C132, C133, C15, C16, C18, C19, C20, C33, C47, C54, C55, C56, C57, C58, C59, C60, C61, C62, C63, C64, C65, C66, C79, C80, C81, C82, C83, C84, C85, C86, C87, C88, C89, C90, C97, C98, C99: moved to B.Cu
- moved R8 256.3 mm to (117.8, 32.2), turned to 180 degrees
- moved U6 250.0 mm to (118.0, 37.5)
- moved C110 242.9 mm to (201.3, 155.9), turned to -90 degrees
- moved C47 239.5 mm to (150.0, 111.4), turned to 180 degrees
- moved TP3 237.0 mm to (167.9, 37.5)
- moved TP1 224.6 mm to (171.9, 52.0)
- moved C20 223.5 mm to (193.0, 97.7), turned to 180 degrees
- moved U7 222.8 mm to (196.6, 92.4)
- moved CR2 221.1 mm to (197.3, 46.7), turned to 180 degrees
- moved TP6 220.0 mm to (149.8, 41.6)
- moved TP14 218.2 mm to (206.9, 102.6)
- moved CR1 210.8 mm to (142.9, 55.8), turned to 90 degrees
- moved TP2 207.6 mm to (136.6, 57.9)
- moved TP13 206.2 mm to (187.9, 104.6)
- moved TP7 206.1 mm to (115.5, 45.7)
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