File: ExoFlexV2/blockdiagram.kicad_sch (KiCad schematic)
At the start: 0 parts

Commit message: Finalisation 1
- Ajout de pages pour la gestion des signaux négatif
- Modification des pages de torque et amplitude
Other:
- note added: "10xRes1k : 5V @ 50mA Total current : 5V @ 50mA"
- note added: "12xOrGate : 5V @ 384,12mA Total current : 5V @ 385mA"
- note added: "1xOrGate : 5V @ 32,01mA 3xANDGate : 5V @ 96,03mA 4xNOTGte : 5V @ 130mA 2x200k : 5V 0,050mA Total current : 5V @ 260mA"
- note added: "24V NUM : 105mA - 2,52W 5V NUM :"
- note added: "2xANDGate : 5V @ 64,02mA 4xNOTGte : 5V @ 128,04mA 3x200k : 5V @ 0,075mA 3x10k : 5V @ 1,5mA Total current : 5V @ 195mA"
- note added: "2xComp : 5VA @ 11mA 2xORGate : 5V @ 64,02mA 3xPot1k : 5VA @ 15mA Total current : 5V @ 65mA 5VA @ 28mA"
- note added: "2xMUX8_1 : 5V @ 100mA Total current : 5V @ 100mA"
- note added: "2xOrGate : 5V @ 64,02mA 7xNOTGte : 5V @ 224,07mA 7x10k : 5V @ 3,5mA 3x200k : 5V @ 0,075mA Total current : 5VA @ 295mA"
- note added: "3xComp : 5VA @ 16,5mA 2xANDGate : 5V @ 64,02mA 1xNOTGte : 5V @ 32,01mA 3xPot1k : 5VA @ 15mA 3x200k : 5V @ 0,075mA Total current : 5V @ 100mA 5VA @ 32mA"
- note added: "3xComp : 5VA @ 16,5mA 2xANDGate : 5V @ 64,02mA 1xNOTGte : 5V @ 32,01mA 3xPot1k : 5VA @ 15mA Total current : 5V @ 115mA 5VA @ 16,5mA"
- note added: "3xComp : 5VA @ 16,5mA 2xOrGate : 5V @ 64,02mA 3xPullUp : 5V @ 0,075mA 3xPot10k : 5VA @ 1,5mA 3xLimit : 5VA @ 1,47mA 3x910k : 5VA @ 0,016mA 6x200k : 5VA @ 0,15mA Total current : 5V @ 90mA"
- note added: "3xComp : 5VA @ 24,5mA 2xOrGate : 5V @ 64,02mA 3xInstAmp : ±5VA @ 150,9mA 3xPot10k : 5VA @ 1,5mA 3xLim10,2k : 5VA @ 1,47mA 3x200k : 5V @ 0,075mA 3x910k: 5VA @ 0,016mA Total current : 5VA @ 180mA -5VA @ 152mA 5V @150,02mA"
- note added: "3xRes1k : 5V @ 15mA 3xRes100k : 5V @ 0,15mA 3xRes5,1k : 5V @ 2,94mA 3xLC : 5V @ 15mA Total current : 5V @ 35mA"
- note added: "4xANDGate : 5V @ 128,04mA 7xNOTGate : 5V @ 224,07mA 6x200k : 5V @0,15mA 4x10k : 5V @ 2mA Total current : 5V @ 360mA"
- note added: "4xRes1k : 5V @ 20mA 2xEmittor : 5VA @ 200mA 2xReceptor : 5VA @ 100mA 4xRes100k : 5V @ 0,2mA 2xRes68 : 5V @ 147mA 2xRes 150 : 5V @ 66,6mA Total current : 5V @ 535mA"
- note added: "5xMagEncoder : 5VA @ 32,5mA 3xTorSensor : ±5VA @ 20,55mA Total current : 5VA @ 54mA -5VA @ 22mA"
- note added: "5xORGate : 5V @ 160,05mA 6x100k : 5V @ 0,3mA 6x200k : 5V @ 0,15mA Total current : 5V @ 162mA"
- note added: "5xORGate : 5V @ 160,05mA 7x100k : 5V @ 0,35mA 7x200k : 5V @ 0,175mA Total current : 5V @ 162mA"
- note added: "6xNOTGate : 5V @ 192,06mA 3xANDGate : 5V @ 96,03mA 3xORGate : 5V @ 96,03mA 4xMUX8_1 : 5v @ 150mA Total current : 5V @ 540mA"
- note added: "Bus Adapter : 5V @ 75mA 2xTempSensor : N/A (uA) Total current : 5V @ 75mA"
- note added: "Contacteur : 24V @ 100mA CoilRelais : 5V @ 20mA FreeWheel5V : 5V @ 2mA FreeWheel24V : 24V @ 4,16mA Latch : 5V @ 1mA Total Current : 5V @ 25 mA 24V @ 105mA"
- note added: "STM32 : 5V @ 500mA PI5 : 5V @ 5A Total Current : 5V @ 5,5A"
