File: 1-ExoFlexV2/_autosave-ExoFlex_Kicad.kicad_pcb (KiCad board)
At the start: 4 copper layers, 360 x 226 mm, 975 parts, among them J1 14 AWG, J10 SSW-115-01-G-D, J100 Jumper, J101 Jumper, J102 Jumper, J103 Jumper, J104 Jumper, J105 Jumper, J106 Jumper, J107 Jumper, J108 Jumper, J109 Jumper, J11 SSW-110-01-G-D, J110 Jumper, J111 Jumper, J112 Jumper, J113 Jumper, J114 Jumper, J115 Jumper, J116 Jumper, J117 Jumper, J118 Jumper, J119 Jumper, J12 SSW-117-01-G-D, J120 Jumper, J121 Jumper, J122 Jumper, J123 Jumper, J124 Jumper, J125 Jumper, J126 Jumper, J127 Jumper, J128 Jumper, J129 Jumper, J13 3, J130 Jumper, J131 Jumper, J14 3, J15 3, J16 5, J17 5, J18 5, J19 3, J2 Jumper, J20 3, J21 3, J22 3, J23 3, J24 3, J25 2, J26 2, J27 2, J28 2, J29 2, J3 14 AWG, J30 2, J31 2, J32 2, J33 2, J34 2, J35 2, J36 2, J37 2, J38 2, J39 4, J4 14 AWG, J40 4, J41 4, J42 4, J43 Jumper, J44 Jumper, J45 Jumper, J46 Jumper, J47 3, J48 3, J49 3, J5 Jumper, J50 2, J51 2, J52 2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

Commit message: Bug NetList
- Ajout de net-tie pour les GND et et les +5V
Connections:
- net DOR_AMP_INT renamed EXT_AMP_INT
