File: 1-ExoFlexV2/powersecurity.kicad_sch (KiCad schematic)
At the start: 25 parts, among them J1 14 AWG, J2 Jumper, J3 14 AWG, J4 14 AWG, K1 Relay, Q1 MOSFET 20V 200mA, U1 TVS 24V, U2 Shott 100V, U3 Inverter, U4 SR-Latch

Commit message: PLacement 2
- Puissance
- signaux
-
Parts:
- removed J4: 14 AWG, FootPrintLib:PHOENIX_1755736, symbol SymLib:1729128
- removed TP4: TestPoint, FootPrint:KEYSTONE_5005, symbol SymLib:5005
Other:
- note removed: "OutPut 5V sécurité"
Changed lines of the file:
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@@
   (junction (at 64.77 72.39) (diameter 0) (color 0 0 0 0)
   )
-  (junction (at 217.17 96.52) (diameter 0) (color 0 0 0 0)
-  )
   (junction (at 44.45 74.93) (diameter 0) (color 0 0 0 0)
   )
@@
   )
   (junction (at 96.52 49.53) (diameter 0) (color 0 0 0 0)
-  )
-  (junction (at 203.2 96.52) (diameter 0) (color 0 0 0 0)
   )
   (junction (at 30.48 127) (diameter 0) (color 0 0 0 0)
@@
   (no_connect (at 146.05 121.92))
   (no_connect (at 146.05 124.46))
-  (wire (pts (xy 107.95 124.46) (xy 123.19 124.46))
+  (wire (pts (xy 115.57 124.46) (xy 123.19 124.46))
     (stroke (width 0) (type default) (color 0 0 0 0))
   )
@@
     (stroke (width 0) (type default) (color 0 0 0 0))
   )
-  (wire (pts (xy 245.11 99.06) (xy 245.11 100.33))
-    (stroke (width 0) (type default) (color 0 0 0 0))
-  )
   (wire (pts (xy 157.48 52.07) (xy 143.51 52.07))
     (stroke (width 0) (type default) (color 0 0 0 0))
@@
   (wire (pts (xy 186.69 49.53) (xy 195.072 48.768))
     (stroke (width 0) (type default) (color 0 0 0 0))
-  )
-  (polyline (pts (xy 234.95 80.01) (xy 234.95 106.68))
-    (stroke (width 0.25) (type solid) (color 0 0 0 0))
   )
   (wire (pts (xy 172.72 127) (xy 181.61 127))
@@
     (stroke (width 0) (type default) (color 0 0 0 0))
   )
-  (wire (pts (xy 203.2 96.52) (xy 217.17 96.52))
-    (stroke (width 0) (type default) (color 0 0 0 0))
-  )
   (wire (pts (xy 143.51 46.99) (xy 143.51 52.07))
     (stroke (width 0) (type default) (color 0 0 0 0))
@@
     (stroke (width 0.5) (type dash) (color 37 168 45 1))
   )
-  (wire (pts (xy 217.17 96.52) (xy 252.73 96.52))
-    (stroke (width 0) (type default) (color 0 0 0 0))
-  )
   (wire (pts (xy 74.93 127) (xy 85.09 127))
     (stroke (width 0) (type default) (color 0 0 0 0))
@@
     (stroke (width 0) (type default) (color 0 0 0 0))
   )
-  (wire (pts (xy 203.2 80.01) (xy 203.2 96.52))
-    (stroke (width 0) (type default) (color 0 0 0 0))
-  )
-  (wire (pts (xy 252.73 99.06) (xy 245.11 99.06))
+  (wire (pts (xy 203.2 80.01) (xy 203.2 123.19))
     (stroke (width 0) (type default) (color 0 0 0 0))
   )
@@
     (stroke (width 0) (type default) (color 0 0 0 0))
   )
-  (wire (pts (xy 203.2 96.52) (xy 203.2 123.19))
-    (stroke (width 0) (type default) (color 0 0 0 0))
-  )
   (wire (pts (xy 96.52 69.85) (xy 96.52 76.2))
     (stroke (width 0) (type default) (color 0 0 0 0))
@@
     (stroke (width 0) (type default) (color 0 0 0 0))
   )
-  (polyline (pts (xy 234.95 80.01) (xy 280.67 80.01))
-    (stroke (width 0.25) (type solid) (color 0 0 0 0))
-  )
   (polyline (pts (xy 173.99 168.91) (xy 173.99 195.58))
     (stroke (width 0.25) (type solid) (color 0 0 0 0))
@@
     (stroke (width 0) (type default) (color 0 0 0 0))
   )
-  (polyline (pts (xy 280.67 106.68) (xy 234.95 106.68))
-    (stroke (width 0.25) (type solid) (color 0 0 0 0))
-  )
   (wire (pts (xy 34.29 74.93) (xy 44.45 74.93))
     (stroke (width 0) (type default) (color 0 0 0 0))
@@
   )
   (polyline (pts (xy 278.13 33.02) (xy 278.13 59.69))
-    (stroke (width 0.25) (type solid) (color 0 0 0 0))
-  )
-  (polyline (pts (xy 280.67 80.01) (xy 280.67 106.68))
     (stroke (width 0.25) (type solid) (color 0 0 0 0))
   )
@@
     (effects (font (size 2.5 2.5) (thickness 0.5) bold) (justify left bottom))
   )
-  (text "OutPut 5V sécurité" (at 238.76 85.09 0)
-    (effects (font (size 2.5 2.5) (thickness 0.5) bold) (justify left bottom))
-  )
   (text "Contacteur : 24V @ 100mA\nCoilRelais : 5V @ 20mA\nFreeWheel5V : 5V @ 2mA\nFreeWheel24V : 24V @ 4,16mA\nLatch : 5V @ 1mA\n\nTotal Current : 5V @ 25,2 mA\n		    24V @ 109,37mA"
     (at 224.79 161.29 0)
     (effects (font (size 2.25 2.25) (thickness 0.45) bold) (justify left bottom))
   )
-  (global_label "ALIM_SEC" (shape input) (at 107.95 124.46 180) (fields_autoplaced)
+  (global_label "ALIM_SEC" (shape input) (at 115.57 124.46 180) (fields_autoplaced)
     (effects (font (size 1.27 1.27) (thickness 0.254) bold) (justify right))
-    (property "Intersheet References" "${INTERSHEET_REFS}" (id 0) (at 96.387 124.587 0)
+    (property "Intersheet References" "${INTERSHEET_REFS}" (id 0) (at 104.007 124.587 0)
       (effects (font (size 1.27 1.27) (thickness 0.254) bold) (justify right) hide)
     )
@@
     (pin "3")
   )
-  (symbol (lib_id "SymLib:5005") (at 217.17 91.44 90) (unit 1)
-    (in_bom yes) (on_board yes)
-    (property "Reference" "TP4" (id 0) (at 215.9 88.9 90)
-      (effects (font (size 1.27 1.27)) (justify right))
-    )
-    (property "Value" "TestPoint" (id 1) (at 213.36 99.06 90)
-      (effects (font (size 1.27 1.27)) (justify right))
-    )
-    (property "Footprint" "FootPrint:KEYSTONE_5005" (id 2) (at 217.17 91.44 0)
-      (effects (font (size 1.27 1.27)) (justify bottom) hide)
-    )
-    (property "Datasheet" "~" (id 3) (at 217.17 91.44 0)
-      (effects (font (size 1.27 1.27)) hide)
-    )
-    (property "MF" "Keystone Electronics" (id 4) (at 217.17 91.44 0)
-      (effects (font (size 1.27 1.27)) (justify bottom) hide)
-    )
-    (property "DESCRIPTION" "PC TEST POINT COMPACT RED" (id 5) (at 217.17 91.44 0)
-      (effects (font (size 1.27 1.27)) (justify bottom) hide)
-    )
-    (property "PACKAGE" "0.125\" Dia x 0.220\" L " (id 6) (at 217.17 91.44 0)
-      (effects (font (size 1.27 1.27)) (justify bottom) hide)
-    )
-    (property "PRICE" "None" (id 7) (at 217.17 91.44 0)
-      (effects (font (size 1.27 1.27)) (justify bottom) hide)
-    )
-    (property "MP" "5005" (id 8) (at 217.17 91.44 0)
-      (effects (font (size 1.27 1.27)) (justify bottom) hide)
-    )
-    (property "AVAILABILITY" "In Stock" (id 9) (at 217.17 91.44 0)
-      (effects (font (size 1.27 1.27)) (justify bottom) hide)
-    )
-    (property "PURCHASE-URL" "" (id 10) (at 217.17 91.44 0)
-      (effects (font (size 1.27 1.27)) (justify bottom) hide)
-    )
-    (property "MANUFACTURER" "Keystone Electronics" (id 11) (at 217.17 91.44 0)
-      (effects (font (size 1.27 1.27)) hide)
-    )
-    (property "PART NUMBER" "5005" (id 12) (at 217.17 91.44 0)
-      (effects (font (size 1.27 1.27)) hide)
-    )
-    (property "TYPE" "Through Hole" (id 13) (at 217.17 91.44 0)
-      (effects (font (size 1.27 1.27)) hide)
-    )
-    (property "NOTES" "DO NOT POPULATE" (id 14) (at 217.17 91.44 0)
-      (effects (font (size 1.27 1.27)) hide)
-    )
-    (pin "TP")
-  )
   (symbol (lib_id "power:GND") (at 205.74 133.35 0) (unit 1)
     (in_bom yes) (on_board yes) (fields_autoplaced)
@@
     (pin "6")
   )
-  (symbol (lib_id "power:GND") (at 245.11 100.33 0) (unit 1)
-    (in_bom yes) (on_board yes) (fields_autoplaced)
-    (property "Reference" "#PWR018" (id 0) (at 245.11 106.68 0)
-      (effects (font (size 1.27 1.27)) hide)
-    )
-    (property "Value" "GND" (id 1) (at 245.11 105.41 0))
-    (property "Footprint" "" (id 2) (at 245.11 100.33 0)
-      (effects (font (size 1.27 1.27)) hide)
-    )
-    (property "Datasheet" "" (id 3) (at 245.11 100.33 0)
-      (effects (font (size 1.27 1.27)) hide)
-    )
-    (pin "1")
-  )
   (symbol (lib_id "power:+5V") (at 148.59 119.38 0) (unit 1)
     (in_bom yes) (on_board yes) (fields_autoplaced)
@@
     (pin "3")
   )
-  (symbol (lib_id "SymLib:1729128") (at 250.19 96.52 0) (unit 1)
-    (in_bom yes) (on_board yes)
-    (property "Reference" "J4" (id 0) (at 255.27 91.44 0)
-      (effects (font (size 1.524 1.524)) (justify left))
-    )
-    (property "Value" "14 AWG" (id 1) (at 254 102.87 0)
-      (effects (font (size 1.524 1.524)) (justify left))
-    )
-    (property "Footprint" "FootPrintLib:PHOENIX_1755736" (id 2) (at 252.73 87.63 0)
-      (effects (font (size 1.27 1.27) italic) hide)
-    )
-    (property "Datasheet" "1755736" (id 3) (at 245.11 88.9 0)
-      (effects (font (size 1.27 1.27) italic) hide)
-    )
-    (property "DESCRIPTION" "2 Position Terminal Block Header, Male Pins, Shrouded (4 Side) 0.200\" (5.08mm) Vertical Through Hole" (id 4) (at 250.19 96.52 0)
-      (effects (font (size 1.27 1.27)) hide)
-    )
-    (property "MANUFACTURER" "Phoenix Contact" (id 5) (at 250.19 96.52 0)
-      (effects (font (size 1.27 1.27)) hide)
-    )
-    (property "PACKAGE" "2 POS 0.200\" (5.08mm)" (id 6) (at 250.19 96.52 0)
-      (effects (font (size 1.27 1.27)) hide)
-    )
-    (property "PART NUMBER" "1755736" (id 7) (at 250.19 96.52 0)
-      (effects (font (size 1.27 1.27)) hide)
-    )
-    (property "TYPE" "Through Hole" (id 8) (at 250.19 96.52 0)
-      (effects (font (size 1.27 1.27)) hide)
-    )
-    (pin "1")
-    (pin "2")
-  )
   (symbol (lib_id "Device:R_Small_US") (at 96.52 58.42 180) (unit 1)
