File: 1-ExoFlexV2/conn_proximity.kicad_sch (KiCad schematic)
At the start: 32 parts, among them J35 2POS, J36 2POS, J37 2POS, J38 2POS, J39 4POS, J40 4POS, J41 4POS, J42 4POS

Commit message: Routage 3
- Routage des connecteurs terminé
- Routage des signaux terminé
Parts:
- removed D71, D73: TVS, FootPrint:DPY2_TEX, symbol Device:D_Zener
Connections:
- net EMI_PROX1 is gone; now on net GND: J39.2 (02)
- net EMI_PROX2 is gone; now on net GND: J41.2 (02)
Changed lines of the file:
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@@
 (kicad_sch (version 20211123) (generator eeschema)
   (paper "A4")
-  (junction (at 107.95 133.35) (diameter 0) (color 0 0 0 0)
+  (junction (at 101.6 43.18) (diameter 0) (color 0 0 0 0)
   )
   (junction (at 115.57 81.28) (diameter 0) (color 0 0 0 0)
   )
-  (junction (at 115.57 40.64) (diameter 0) (color 0 0 0 0)
-  )
   (junction (at 101.6 133.35) (diameter 0) (color 0 0 0 0)
   )
   (junction (at 107.95 156.21) (diameter 0) (color 0 0 0 0)
   )
-  (junction (at 107.95 54.61) (diameter 0) (color 0 0 0 0)
-  )
   (junction (at 101.6 173.99) (diameter 0) (color 0 0 0 0)
   )
@@
   (junction (at 107.95 93.98) (diameter 0) (color 0 0 0 0)
   )
-  (junction (at 115.57 120.65) (diameter 0) (color 0 0 0 0)
-  )
   (junction (at 107.95 115.57) (diameter 0) (color 0 0 0 0)
   )
@@
   )
   (junction (at 101.6 93.98) (diameter 0) (color 0 0 0 0)
+  )
+  (junction (at 101.6 123.19) (diameter 0) (color 0 0 0 0)
   )
   (junction (at 115.57 161.29) (diameter 0) (color 0 0 0 0)
@@
     (stroke (width 0) (type default) (color 0 0 0 0))
   )
-  (wire (pts (xy 115.57 120.65) (xy 99.06 120.65))
+  (wire (pts (xy 101.6 120.65) (xy 99.06 120.65))
     (stroke (width 0) (type default) (color 0 0 0 0))
   )
@@
     (stroke (width 0) (type default) (color 0 0 0 0))
   )
-  (wire (pts (xy 115.57 40.64) (xy 115.57 46.99))
+  (wire (pts (xy 101.6 40.64) (xy 101.6 43.18))
     (stroke (width 0) (type default) (color 0 0 0 0))
   )
@@
     (stroke (width 0) (type default) (color 0 0 0 0))
   )
-  (wire (pts (xy 124.46 120.65) (xy 115.57 120.65))
-    (stroke (width 0) (type default) (color 0 0 0 0))
-  )
-  (wire (pts (xy 101.6 133.35) (xy 107.95 133.35))
-    (stroke (width 0) (type default) (color 0 0 0 0))
-  )
-  (wire (pts (xy 115.57 40.64) (xy 99.06 40.64))
-    (stroke (width 0) (type default) (color 0 0 0 0))
-  )
-  (wire (pts (xy 107.95 133.35) (xy 115.57 133.35))
+  (wire (pts (xy 101.6 40.64) (xy 99.06 40.64))
+    (stroke (width 0) (type default) (color 0 0 0 0))
+  )
+  (wire (pts (xy 107.95 133.35) (xy 101.6 133.35))
     (stroke (width 0) (type default) (color 0 0 0 0))
   )
@@
     (stroke (width 0) (type default) (color 0 0 0 0))
   )
-  (wire (pts (xy 124.46 40.64) (xy 115.57 40.64))
-    (stroke (width 0) (type default) (color 0 0 0 0))
-  )
   (wire (pts (xy 101.6 54.61) (xy 107.95 54.61))
     (stroke (width 0) (type default) (color 0 0 0 0))
@@
     (stroke (width 0) (type default) (color 0 0 0 0))
   )
-  (wire (pts (xy 107.95 54.61) (xy 115.57 54.61))
-    (stroke (width 0) (type default) (color 0 0 0 0))
-  )
   (wire (pts (xy 34.29 146.05) (xy 44.45 146.05))
     (stroke (width 0) (type default) (color 0 0 0 0))
@@
     (stroke (width 0) (type default) (color 0 0 0 0))
   )
-  (wire (pts (xy 115.57 120.65) (xy 115.57 125.73))
+  (wire (pts (xy 101.6 120.65) (xy 101.6 123.19))
     (stroke (width 0) (type default) (color 0 0 0 0))
   )
@@
     )
   )
-  (global_label "EMI_PROX1" (shape input) (at 124.46 40.64 0) (fields_autoplaced)
-    (effects (font (size 1.27 1.27) (thickness 0.254) bold) (justify left))
-    (property "Intersheet References" "${INTERSHEET_REFS}" (id 0) (at 137.7164 40.513 0)
-      (effects (font (size 1.27 1.27) (thickness 0.254) bold) (justify left) hide)
-    )
-  )
   (global_label "REC_PROX2_INT" (shape input) (at 120.65 156.21 0) (fields_autoplaced)
     (effects (font (size 1.27 1.27) bold) (justify left))
@@
     )
   )
-  (global_label "EMI_PROX2" (shape input) (at 124.46 120.65 0) (fields_autoplaced)
-    (effects (font (size 1.27 1.27) (thickness 0.254) bold) (justify left))
-    (property "Intersheet References" "${INTERSHEET_REFS}" (id 0) (at 137.7164 120.523 0)
-      (effects (font (size 1.27 1.27) (thickness 0.254) bold) (justify left) hide)
-    )
-  )
   (global_label "BUT_PROX_LEFT1" (shape input) (at 53.34 33.02 0) (fields_autoplaced)
     (effects (font (size 1.27 1.27) (thickness 0.254) bold) (justify left))
@@
     (pin "2")
   )
-  (symbol (lib_id "Device:D_Zener") (at 115.57 50.8 270) (unit 1)
-    (in_bom yes) (on_board yes)
-    (property "Reference" "D71" (id 0) (at 114.3 48.26 90)
-      (effects (font (size 1.27 1.27)) (justify right))
-    )
-    (property "Value" "TVS" (id 1) (at 118.11 53.34 90)
-      (effects (font (size 1.27 1.27)) (justify right))
-    )
-    (property "Footprint" "FootPrint:DPY2_TEX" (id 2) (at 115.57 50.8 0)
-      (effects (font (size 1.27 1.27)) hide)
-    )
-    (property "Datasheet" "~" (id 3) (at 115.57 50.8 0)
-      (effects (font (size 1.27 1.27)) hide)
-    )
-    (property "DESCRIPTION" "TVS DIODE 5.5VWM 14VC 2X1SON" (id 4) (at 115.57 50.8 0)
-      (effects (font (size 1.27 1.27)) hide)
-    )
-    (property "MANUFACTURER" "Texas Instruments" (id 5) (at 115.57 50.8 0)
-      (effects (font (size 1.27 1.27)) hide)
-    )
-    (property "PACKAGE" "0402 (1006 Metric)" (id 6) (at 115.57 50.8 0)
-      (effects (font (size 1.27 1.27)) hide)
-    )
-    (property "PART NUMBER" "TPD1E05U06DPYR" (id 7) (at 115.57 50.8 0)
-      (effects (font (size 1.27 1.27)) hide)
-    )
-    (property "TYPE" "SMD" (id 8) (at 115.57 50.8 0)
-      (effects (font (size 1.27 1.27)) hide)
-    )
-    (pin "1")
-    (pin "2")
-  )
   (symbol (lib_id "power:+5V") (at 49.53 143.51 0) (unit 1)
     (in_bom yes) (on_board yes) (fields_autoplaced)
@@
     (pin "1")
   )
-  (symbol (lib_id "Device:D_Zener") (at 115.57 129.54 270) (unit 1)
-    (in_bom yes) (on_board yes)
-    (property "Reference" "D73" (id 0) (at 114.3 127 90)
-      (effects (font (size 1.27 1.27)) (justify right))
-    )
-    (property "Value" "TVS" (id 1) (at 118.11 132.08 90)
-      (effects (font (size 1.27 1.27)) (justify right))
-    )
-    (property "Footprint" "FootPrint:DPY2_TEX" (id 2) (at 115.57 129.54 0)
-      (effects (font (size 1.27 1.27)) hide)
-    )
-    (property "Datasheet" "~" (id 3) (at 115.57 129.54 0)
-      (effects (font (size 1.27 1.27)) hide)
-    )
-    (property "DESCRIPTION" "TVS DIODE 5.5VWM 14VC 2X1SON" (id 4) (at 115.57 129.54 0)
-      (effects (font (size 1.27 1.27)) hide)
-    )
-    (property "MANUFACTURER" "Texas Instruments" (id 5) (at 115.57 129.54 0)
-      (effects (font (size 1.27 1.27)) hide)
-    )
-    (property "PACKAGE" "0402 (1006 Metric)" (id 6) (at 115.57 129.54 0)
-      (effects (font (size 1.27 1.27)) hide)
-    )
-    (property "PART NUMBER" "TPD1E05U06DPYR" (id 7) (at 115.57 129.54 0)
-      (effects (font (size 1.27 1.27)) hide)
-    )
-    (property "TYPE" "SMD" (id 8) (at 115.57 129.54 0)
-      (effects (font (size 1.27 1.27)) hide)
-    )
-    (pin "1")
-    (pin "2")
-  )
   (symbol (lib_name "1751112_2") (lib_id "SymLib:1751112") (at 88.9 38.1 180) (unit 1)
